File: XC5VLX30T_testboard/XC5VLX30T_testboard.kicad_pcb (KiCad board)
At the start: 2 copper layers, 1 part, among them U1 XC5VLX30T-1FFG665I

Commit message: h
Parts:
- added C1: 220uF, Capacitor_Tantalum_SMD:CP_EIA-3528-12_Kemet-T, F.Cu at (159.5, 99.5)
- added C10: 15nF, Capacitor_Tantalum_SMD:CP_EIA-3528-12_Kemet-T, F.Cu at (213.3, 201.0)
- added C11: 1uF, Capacitor_Tantalum_SMD:CP_EIA-3528-12_Kemet-T, F.Cu at (213.8, 213.5)
- added C12: 470nF, Capacitor_Tantalum_SMD:CP_EIA-3528-12_Kemet-T, F.Cu at (214.3, 192.5)
- added C13: 120pF, Capacitor_Tantalum_SMD:CP_EIA-3528-12_Kemet-T, F.Cu at (192.3, 171.5)
- added C14: 470uF, Capacitor_Tantalum_SMD:CP_EIA-3528-12_Kemet-T, F.Cu at (190.8, 179.0)
- added C15: 220uF, Capacitor_Tantalum_SMD:CP_EIA-3528-12_Kemet-T, F.Cu at (171.8, 209.0)
- added C16: 15nF, Capacitor_Tantalum_SMD:CP_EIA-3528-12_Kemet-T, F.Cu at (180.3, 220.0)
- added C17: 1uF, Capacitor_Tantalum_SMD:CP_EIA-3528-12_Kemet-T, F.Cu at (181.3, 207.0)
- added C18: 470nF, Capacitor_Tantalum_SMD:CP_EIA-3528-12_Kemet-T, F.Cu at (190.3, 190.0)
- added C19: 120pF, Capacitor_Tantalum_SMD:CP_EIA-3528-12_Kemet-T, F.Cu at (190.8, 218.5)
- added C2: 15nF, Capacitor_Tantalum_SMD:CP_EIA-3528-12_Kemet-T, F.Cu at (150.5, 119.0)
- added C20: 470uF, Capacitor_Tantalum_SMD:CP_EIA-3528-12_Kemet-T, F.Cu at (205.8, 215.5)
- added C3: 1uF, Capacitor_Tantalum_SMD:CP_EIA-3528-12_Kemet-T, F.Cu at (150.5, 114.5)
- added C4: 470nF, Capacitor_Tantalum_SMD:CP_EIA-3528-12_Kemet-T, F.Cu at (168.5, 116.5)
- added C5: 120pF, Capacitor_Tantalum_SMD:CP_EIA-3528-12_Kemet-T, F.Cu at (162.0, 124.5)
- added C6: 470uF, Capacitor_Tantalum_SMD:CP_EIA-3528-12_Kemet-T, F.Cu at (177.0, 119.0)
- added C8: 470uF, Capacitor_Tantalum_SMD:CP_EIA-3528-12_Kemet-T, F.Cu at (174.5, 126.0)
- added C9: 220uF, Capacitor_Tantalum_SMD:CP_EIA-3528-12_Kemet-T, F.Cu at (198.3, 203.5)
- added L1: 680nH, Inductor_SMD:L_Coilcraft_XAL7050-XXX, F.Cu at (177.1, 109.0)
- added L2: 680nH, Inductor_SMD:L_Coilcraft_XAL7050-XXX, F.Cu at (195.9, 153.5)
- added L3: 680nH, Inductor_SMD:L_Coilcraft_XAL7050-XXX, F.Cu at (169.3, 194.5)
- added Q1: STP40NF03L, Package_TO_SOT_THT:TO-220-3_Vertical, F.Cu at (150.0, 106.5)
- added Q2: STP40NF03L, Package_TO_SOT_THT:TO-220-3_Vertical, F.Cu at (163.5, 106.4)
- added Q3: STP40NF03L, Package_TO_SOT_THT:TO-220-3_Vertical, F.Cu at (200.8, 188.9)
- added Q4: STP40NF03L, Package_TO_SOT_THT:TO-220-3_Vertical, F.Cu at (202.3, 163.9)
- added Q5: STP40NF03L, Package_TO_SOT_THT:TO-220-3_Vertical, F.Cu at (165.3, 179.5)
- added Q6: STP40NF03L, Package_TO_SOT_THT:TO-220-3_Vertical, F.Cu at (177.8, 194.9)
- added U10: 74ACT245MTC, test_bufferchip_libraryfootprint:TSSOP20_4P4X6P5_ONS, F.Cu at (95.5, 93.5)
- added U11: 74ACT245MTC, test_bufferchip_libraryfootprint:TSSOP20_4P4X6P5_ONS, F.Cu at (95.5, 101.8)
- added U12: 74ACT245MTC, test_bufferchip_libraryfootprint:TSSOP20_4P4X6P5_ONS, F.Cu at (95.5, 110.1)
- added U13: 74ACT245MTC, test_bufferchip_libraryfootprint:TSSOP20_4P4X6P5_ONS, F.Cu at (95.1, 160.9)
- added U14: 74ACT245MTC, test_bufferchip_libraryfootprint:TSSOP20_4P4X6P5_ONS, F.Cu at (95.1, 169.2)
- added U15: 74ACT245MTC, test_bufferchip_libraryfootprint:TSSOP20_4P4X6P5_ONS, F.Cu at (95.1, 177.5)
- added U16: 74ACT245MTC, test_bufferchip_libraryfootprint:TSSOP20_4P4X6P5_ONS, F.Cu at (95.1, 185.7)
- added U17: 74ACT245MTC, test_bufferchip_libraryfootprint:TSSOP20_4P4X6P5_ONS, F.Cu at (95.1, 194.0)
- added U18: 74ACT245MTC, test_bufferchip_libraryfootprint:TSSOP20_4P4X6P5_ONS, F.Cu at (95.0, 202.7)
- added U19: 74ACT245MTC, test_bufferchip_libraryfootprint:TSSOP20_4P4X6P5_ONS, F.Cu at (95.0, 210.9)
- added U2: LM3150MHX/NOPB, lm3150Library:MXA14A, F.Cu at (159.7, 116.5)
- added U20: 74ACT245MTC, test_bufferchip_libraryfootprint:TSSOP20_4P4X6P5_ONS, F.Cu at (95.0, 219.2)
- added U21: 74ACT245MTC, test_bufferchip_libraryfootprint:TSSOP20_4P4X6P5_ONS, F.Cu at (95.0, 227.5)
- added U22: 74ACT245MTC, test_bufferchip_libraryfootprint:TSSOP20_4P4X6P5_ONS, F.Cu at (95.0, 235.7)
- added U23: 74ACT245MTC, test_bufferchip_libraryfootprint:TSSOP20_4P4X6P5_ONS, F.Cu at (95.0, 244.7)
- added U24: 74ACT245MTC, test_bufferchip_libraryfootprint:TSSOP20_4P4X6P5_ONS, F.Cu at (95.0, 253.0)
- added U25: 74ACT245MTC, test_bufferchip_libraryfootprint:TSSOP20_4P4X6P5_ONS, F.Cu at (95.0, 261.3)
- added U26: 74ACT245MTC, test_bufferchip_libraryfootprint:TSSOP20_4P4X6P5_ONS, F.Cu at (95.0, 269.5)
- added U27: 74ACT245MTC, test_bufferchip_libraryfootprint:TSSOP20_4P4X6P5_ONS, F.Cu at (95.0, 277.8)
- added U28: LM3150MHX/NOPB, lm3150Library:MXA14A, F.Cu at (204.8, 178.5)
- added U29: LM3150MHX/NOPB, lm3150Library:MXA14A, F.Cu at (180.3, 185.0)
- added U3: 74ACT245MTC, test_bufferchip_libraryfootprint:TSSOP20_4P4X6P5_ONS, F.Cu at (95.3, 118.9)
- added U30: 74ACT245PC, 16DIP_74ACT:PDIP20_26P42X6P6_ONS, F.Cu at (306.8, 115.8)
- added U31: 74ACT245PC, 16DIP_74ACT:PDIP20_26P42X6P6_ONS, F.Cu at (308.5, 193.6)
- added U32: 74ACT245PC, 16DIP_74ACT:PDIP20_26P42X6P6_ONS, F.Cu at (308.7, 271.8)
- added U33: 74ACT245PC, 16DIP_74ACT:PDIP20_26P42X6P6_ONS, F.Cu at (302.1, 90.7)
- added U34: 74ACT245PC, 16DIP_74ACT:PDIP20_26P42X6P6_ONS, F.Cu at (358.1, 65.7)
- added U35: 74ACT245PC, 16DIP_74ACT:PDIP20_26P42X6P6_ONS, F.Cu at (357.8, 147.8)
- added U36: 74ACT245PC, 16DIP_74ACT:PDIP20_26P42X6P6_ONS, F.Cu at (357.1, 231.0)
- added U37: 74ACT245PC, 16DIP_74ACT:PDIP20_26P42X6P6_ONS, F.Cu at (357.6, 316.5)
- added U38: 74ACT245PC, 16DIP_74ACT:PDIP20_26P42X6P6_ONS, F.Cu at (358.9, 372.9)
- added U39: 74ACT245PC, 16DIP_74ACT:PDIP20_26P42X6P6_ONS, F.Cu at (308.3, 140.8)
- added U4: 74ACT245MTC, test_bufferchip_libraryfootprint:TSSOP20_4P4X6P5_ONS, F.Cu at (95.3, 127.1)
- added U40: 74ACT245PC, 16DIP_74ACT:PDIP20_26P42X6P6_ONS, F.Cu at (308.3, 218.3)
- added U41: 74ACT245PC, 16DIP_74ACT:PDIP20_26P42X6P6_ONS, F.Cu at (308.7, 299.9)
- added U42: 74ACT245PC, 16DIP_74ACT:PDIP20_26P42X6P6_ONS, F.Cu at (301.9, 64.9)
- added U43: 74ACT245PC, 16DIP_74ACT:PDIP20_26P42X6P6_ONS, F.Cu at (358.1, 93.8)
- added U44: 74ACT245PC, 16DIP_74ACT:PDIP20_26P42X6P6_ONS, F.Cu at (357.8, 175.9)
- added U45: 74ACT245PC, 16DIP_74ACT:PDIP20_26P42X6P6_ONS, F.Cu at (357.1, 259.1)
- added U46: 74ACT245PC, 16DIP_74ACT:PDIP20_26P42X6P6_ONS, F.Cu at (357.6, 344.6)
- added U47: 74ACT245PC, 16DIP_74ACT:PDIP20_26P42X6P6_ONS, F.Cu at (351.6, 35.7)
- added U48: 74ACT245PC, 16DIP_74ACT:PDIP20_26P42X6P6_ONS, F.Cu at (308.5, 167.1)
- added U49: 74ACT245PC, 16DIP_74ACT:PDIP20_26P42X6P6_ONS, F.Cu at (308.3, 244.3)
- added U5: 74ACT245MTC, test_bufferchip_libraryfootprint:TSSOP20_4P4X6P5_ONS, F.Cu at (95.3, 135.4)
- added U50: 74ACT245PC, 16DIP_74ACT:PDIP20_26P42X6P6_ONS, F.Cu at (308.7, 327.9)
- added U51: 74ACT245PC, 16DIP_74ACT:PDIP20_26P42X6P6_ONS, F.Cu at (308.6, 355.0)
- added U52: 74ACT245PC, 16DIP_74ACT:PDIP20_26P42X6P6_ONS, F.Cu at (358.1, 121.8)
- added U53: 74ACT245PC, 16DIP_74ACT:PDIP20_26P42X6P6_ONS, F.Cu at (357.8, 204.0)
- added U54: 74ACT245PC, 16DIP_74ACT:PDIP20_26P42X6P6_ONS, F.Cu at (357.1, 287.2)
- added U6: 74ACT245MTC, test_bufferchip_libraryfootprint:TSSOP20_4P4X6P5_ONS, F.Cu at (95.3, 143.6)
- added U7: 74ACT245MTC, test_bufferchip_libraryfootprint:TSSOP20_4P4X6P5_ONS, F.Cu at (95.3, 151.9)
- added U8: 74ACT245MTC, test_bufferchip_libraryfootprint:TSSOP20_4P4X6P5_ONS, F.Cu at (95.5, 77.0)
- added U9: 74ACT245MTC, test_bufferchip_libraryfootprint:TSSOP20_4P4X6P5_ONS, F.Cu at (95.5, 85.3)
- U1: value XC5VLX30T-1FFG665I -> XC5VLX30T-1FFG665C; footprint Library:665-FBGA_XIL -> Library:digikey665-FBGA_XIL
- moved U1 55.5 mm to (163.0, 147.5)
Connections:
- U1 pad A11: unconnected-(U1B-GND-PadA11) -> GND
- U1 pad A16: unconnected-(U1B-GND-PadA16) -> GND
- U1 pad A2: unconnected-(U1A-GND-PadA2) -> GND
- U1 pad A21: unconnected-(U1B-GND-PadA21) -> GND
- U1 pad A26: unconnected-(U1B-GND-PadA26) -> GND
- U1 pad A6: unconnected-(U1A-GND-PadA6) -> GND
- U1 pad AA11: unconnected-(U1F-GND-PadAA11) -> GND
- U1 pad AA16: unconnected-(U1F-VCCO_2-PadAA16) -> VCCO
- U1 pad AA21: unconnected-(U1G-GND-PadAA21) -> GND
- U1 pad AA26: unconnected-(U1G-GND-PadAA26) -> GND
- U1 pad AA4: unconnected-(U1C-GND-PadAA4) -> GND
- U1 pad AB13: unconnected-(U1G-VCCO_4-PadAB13) -> VCCO
- U1 pad AB18: unconnected-(U1G-GND-PadAB18) -> GND
- U1 pad AB2: unconnected-(U1C-GND-PadAB2) -> GND
- U1 pad AB23: unconnected-(U1G-VCCO_17-PadAB23) -> VCCO
- U1 pad AB8: unconnected-(U1C-GND-PadAB8) -> GND
- U1 pad AC10: unconnected-(U1G-VCCO_18-PadAC10) -> VCCO
- U1 pad AC15: unconnected-(U1G-GND-PadAC15) -> GND
- U1 pad AC2: unconnected-(U1C-GND-PadAC2) -> GND
- U1 pad AC20: unconnected-(U1G-VCCO_17-PadAC20) -> VCCO
- U1 pad AC25: unconnected-(U1G-GND-PadAC25) -> GND
- U1 pad AC5: unconnected-(U1C-GND-PadAC5) -> GND
- U1 pad AD12: unconnected-(U1G-GND-PadAD12) -> GND
- U1 pad AD17: unconnected-(U1G-VCCO_2-PadAD17) -> VCCO
- U1 pad AD22: unconnected-(U1G-GND-PadAD22) -> GND
- U1 pad AE14: unconnected-(U1G-VCCO_4-PadAE14) -> VCCO
- U1 pad AE19: unconnected-(U1G-GND-PadAE19) -> GND
- U1 pad AE24: unconnected-(U1G-VCCO_17-PadAE24) -> VCCO
- U1 pad AE4: unconnected-(U1C-GND-PadAE4) -> GND
- U1 pad AE9: unconnected-(U1C-GND-PadAE9) -> GND
- U1 pad AF11: unconnected-(U1G-GND-PadAF11) -> GND
- U1 pad AF16: unconnected-(U1G-GND-PadAF16) -> GND
- U1 pad AF2: unconnected-(U1C-GND-PadAF2) -> GND
- U1 pad AF21: unconnected-(U1G-GND-PadAF21) -> GND
- U1 pad AF26: unconnected-(U1G-GND-PadAF26) -> GND
- U1 pad AF6: unconnected-(U1C-GND-PadAF6) -> GND
- U1 pad B18: unconnected-(U1C-GND-PadB18) -> GND
- U1 pad B8: unconnected-(U1A-GND-PadB8) -> GND
- U1 pad C15: unconnected-(U1C-GND-PadC15) -> GND
- U1 pad C20: unconnected-(U1C-GND-PadC20) -> GND
- U1 pad C25: unconnected-(U1C-GND-PadC25) -> GND
- U1 pad C4: unconnected-(U1A-GND-PadC4) -> GND
- U1 pad C5: unconnected-(U1A-GND-PadC5) -> GND
- U1 pad D12: unconnected-(U1C-GND-PadD12) -> GND
- U1 pad D2: unconnected-(U1A-GND-PadD2) -> GND
- U1 pad D22: unconnected-(U1D-GND-PadD22) -> GND
- U1 pad E19: unconnected-(U1D-GND-PadE19) -> GND
- U1 pad E2: unconnected-(U1A-GND-PadE2) -> GND
- U1 pad E9: unconnected-(U1A-GND-PadE9) -> GND
- U1 pad F16: unconnected-(U1D-GND-PadF16) -> GND
- U1 pad F26: unconnected-(U1D-GND-PadF26) -> GND
- U1 pad F4: unconnected-(U1A-GND-PadF4) -> GND
- U1 pad F6: unconnected-(U1A-GND-PadF6) -> GND
- U1 pad G13: unconnected-(U1D-GND-PadG13) -> GND
- U1 pad G23: unconnected-(U1D-GND-PadG23) -> GND
- U1 pad H10: unconnected-(U1D-GND-PadH10) -> GND
- U1 pad H14: unconnected-(U1D-GND-PadH14) -> GND
- U1 pad H15: unconnected-(U1D-VCCINT-PadH15) -> VccINT
- U1 pad H16: unconnected-(U1D-GND-PadH16) -> GND
- U1 pad H17: unconnected-(U1D-VCCINT-PadH17) -> VccINT
- U1 pad H20: unconnected-(U1D-GND-PadH20) -> GND
- U1 pad J13: unconnected-(U1D-GND-PadJ13) -> GND
- U1 pad J14: unconnected-(U1D-VCCINT-PadJ14) -> VccINT
- U1 pad J15: unconnected-(U1D-GND-PadJ15) -> GND
- U1 pad J16: unconnected-(U1D-VCCINT-PadJ16) -> VccINT
- U1 pad J17: unconnected-(U1D-GND-PadJ17) -> GND
- U1 pad J18: unconnected-(U1D-VCCINT-PadJ18) -> VccINT
- U1 pad J4: unconnected-(U1A-GND-PadJ4) -> GND
- U1 pad J7: unconnected-(U1A-GND-PadJ7) -> GND
- U1 pad K10: unconnected-(U1D-GND-PadK10) -> GND
- U1 pad K12: unconnected-(U1D-GND-PadK12) -> GND
- U1 pad K14: unconnected-(U1E-GND-PadK14) -> GND
- U1 pad K15: unconnected-(U1E-VCCINT-PadK15) -> VccINT
- U1 pad K16: unconnected-(U1E-GND-PadK16) -> GND
- U1 pad K17: unconnected-(U1E-VCCINT-PadK17) -> VccINT
- U1 pad K18: unconnected-(U1E-GND-PadK18) -> GND
- U1 pad K19: unconnected-(U1E-VCCINT-PadK19) -> VccINT
- U1 pad K2: unconnected-(U1A-GND-PadK2) -> GND
- U1 pad K24: unconnected-(U1E-GND-PadK24) -> GND
- U1 pad K9: unconnected-(U1A-VCCAUX-PadK9) -> VccAUX
- U1 pad L10: unconnected-(U1E-VCCINT-PadL10) -> VccINT
- U1 pad L11: unconnected-(U1E-GND-PadL11) -> GND
- U1 pad L12: unconnected-(U1E-VCCINT-PadL12) -> VccINT
- U1 pad L13: unconnected-(U1E-GND-PadL13) -> GND
- U1 pad L14: unconnected-(U1E-VCCINT-PadL14) -> VccINT
- U1 pad L15: unconnected-(U1E-GND-PadL15) -> GND
- U1 pad L16: unconnected-(U1E-VCCINT-PadL16) -> VccINT
- U1 pad L17: unconnected-(U1E-GND-PadL17) -> GND
- U1 pad L18: unconnected-(U1E-VCCINT-PadL18) -> VccINT
- U1 pad L19: unconnected-(U1E-GND-PadL19) -> GND
- U1 pad L2: unconnected-(U1A-GND-PadL2) -> GND
- U1 pad L21: unconnected-(U1E-GND-PadL21) -> GND
- U1 pad L26: unconnected-(U1E-GND-PadL26) -> GND
- U1 pad M10: unconnected-(U1E-GND-PadM10) -> GND
- U1 pad M11: unconnected-(U1E-VCCINT-PadM11) -> VccINT
- U1 pad M12: unconnected-(U1E-GND-PadM12) -> GND
- U1 pad M13: unconnected-(U1E-VCCINT-PadM13) -> VccINT
- U1 pad M16: unconnected-(U1E-GND-PadM16) -> GND
- U1 pad M17: unconnected-(U1E-VCCINT-PadM17) -> VccINT
- U1 pad M18: unconnected-(U1E-GND-PadM18) -> GND
- U1 pad M19: unconnected-(U1E-VCCAUX-PadM19) -> VccAUX
- U1 pad M23: unconnected-(U1E-VCCO_11-PadM23) -> VCCO
- U1 pad M4: unconnected-(U1B-GND-PadM4) -> GND
- U1 pad M8: unconnected-(U1B-GND-PadM8) -> GND
- U1 pad N10: unconnected-(U1E-VCCINT-PadN10) -> VccINT
- U1 pad N11: unconnected-(U1E-GND-PadN11) -> GND
- U1 pad N12: unconnected-(U1E-VCCINT-PadN12) -> VccINT
- U1 pad N13: unconnected-(U1E-GND-PadN13) -> GND
- U1 pad N16: unconnected-(U1E-VCCINT-PadN16) -> VccINT
- U1 pad N17: unconnected-(U1E-GND-PadN17) -> GND
- U1 pad N18: unconnected-(U1E-VCCINT-PadN18) -> VccINT
- U1 pad N19: unconnected-(U1E-GND-PadN19) -> GND
- U1 pad N20: unconnected-(U1E-VCCAUX-PadN20) -> VccAUX
- U1 pad N25: unconnected-(U1E-GND-PadN25) -> GND
- U1 pad N5: unconnected-(U1B-GND-PadN5) -> GND
- U1 pad N9: unconnected-(U1B-GND-PadN9) -> GND
- U1 pad P10: unconnected-(U1E-GND-PadP10) -> GND
- U1 pad P12: unconnected-(U1E-GND-PadP12) -> GND
- U1 pad P13: unconnected-(U1E-VCCINT-PadP13) -> VccINT
- U1 pad P16: unconnected-(U1E-GND-PadP16) -> GND
- U1 pad P17: unconnected-(U1E-VCCINT-PadP17) -> VccINT
- U1 pad P18: unconnected-(U1E-GND-PadP18) -> GND
- U1 pad P19: unconnected-(U1E-VCCAUX-PadP19) -> VccAUX
- U1 pad P22: unconnected-(U1E-GND-PadP22) -> GND
- U1 pad R10: unconnected-(U1E-VCCINT-PadR10) -> VccINT
- U1 pad R11: unconnected-(U1E-GND-PadR11) -> GND
- U1 pad R12: unconnected-(U1E-VCCINT-PadR12) -> VccINT
- U1 pad R13: unconnected-(U1E-GND-PadR13) -> GND
- U1 pad R16: unconnected-(U1E-VCCINT-PadR16) -> VccINT
- U1 pad R17: unconnected-(U1E-GND-PadR17) -> GND
- U1 pad R19: unconnected-(U1E-GND-PadR19) -> GND
- U1 pad R24: unconnected-(U1F-VCCO_13-PadR24) -> VCCO
- U1 pad R4: unconnected-(U1B-GND-PadR4) -> GND
- U1 pad R9: unconnected-(U1B-GND-PadR9) -> GND
- U1 pad T10: unconnected-(U1F-GND-PadT10) -> GND
- U1 pad T11: unconnected-(U1F-VCCINT-PadT11) -> VccINT
- U1 pad T12: unconnected-(U1F-GND-PadT12) -> GND
- U1 pad T13: unconnected-(U1F-VCCINT-PadT13) -> VccINT
- U1 pad T14: unconnected-(U1F-GND-PadT14) -> GND
- U1 pad T15: unconnected-(U1F-VCCINT-PadT15) -> VccINT
- U1 pad T16: unconnected-(U1F-GND-PadT16) -> GND
- U1 pad T17: unconnected-(U1F-VCCINT-PadT17) -> VccINT
- U1 pad T18: unconnected-(U1F-GND-PadT18) -> GND
- U1 pad T19: unconnected-(U1F-VCCAUX-PadT19) -> VccAUX
- U1 pad T2: unconnected-(U1B-GND-PadT2) -> GND
- U1 pad T21: unconnected-(U1F-GND-PadT21) -> GND
- U1 pad T26: unconnected-(U1F-GND-PadT26) -> GND
- U1 pad T6: unconnected-(U1B-GND-PadT6) -> GND
- U1 pad T9: unconnected-(U1B-VCCAUX-PadT9) -> VccAUX
- U1 pad U10: unconnected-(U1F-VCCINT-PadU10) -> VccINT
- U1 pad U11: unconnected-(U1F-GND-PadU11) -> GND
- U1 pad U13: unconnected-(U1F-GND-PadU13) -> GND
- U1 pad U14: unconnected-(U1F-VCCINT-PadU14) -> VccINT
- U1 pad U15: unconnected-(U1F-GND-PadU15) -> GND
- U1 pad U16: unconnected-(U1F-VCCINT-PadU16) -> VccINT
- U1 pad U17: unconnected-(U1F-GND-PadU17) -> GND
- U1 pad U18: unconnected-(U1F-VCCINT-PadU18) -> VccINT
- U1 pad U19: unconnected-(U1F-GND-PadU19) -> GND
- U1 pad U2: unconnected-(U1B-GND-PadU2) -> GND
- U1 pad U23: unconnected-(U1F-GND-PadU23) -> GND
- U1 pad U8: unconnected-(U1B-VCCAUX-PadU8) -> VccAUX
- U1 pad U9: unconnected-(U1B-GND-PadU9) -> GND
- U1 pad V10: unconnected-(U1F-GND-PadV10) -> GND
- U1 pad V14: unconnected-(U1F-GND-PadV14) -> GND
- U1 pad V15: unconnected-(U1F-VCCINT-PadV15) -> VccINT
- U1 pad V16: unconnected-(U1F-GND-PadV16) -> GND
- U1 pad V17: unconnected-(U1F-VCCINT-PadV17) -> VccINT
- U1 pad V18: unconnected-(U1F-GND-PadV18) -> GND
- U1 pad V19: unconnected-(U1F-VCCAUX-PadV19) -> VccAUX
- U1 pad V20: unconnected-(U1F-GND-PadV20) -> GND
- U1 pad V4: unconnected-(U1B-GND-PadV4) -> GND
- U1 pad V5: unconnected-(U1B-GND-PadV5) -> GND
- U1 pad W10: unconnected-(U1F-VCCAUX-PadW10) -> VccAUX
- U1 pad W12: unconnected-(U1F-GND-PadW12) -> GND
- U1 pad W15: unconnected-(U1F-GND-PadW15) -> GND
- U1 pad W17: unconnected-(U1F-GND-PadW17) -> GND
- U1 pad W18: unconnected-(U1F-VCCINT-PadW18) -> VccINT
- U1 pad W19: unconnected-(U1F-GND-PadW19) -> GND
- U1 pad W22: unconnected-(U1F-VCCO_13-PadW22) -> VCCO
- U1 pad W7: unconnected-(U1B-GND-PadW7) -> GND
- U1 pad Y14: unconnected-(U1F-GND-PadY14) -> GND
- U1 pad Y19: unconnected-(U1F-VCCAUX-PadY19) -> VccAUX
- U1 pad Y24: unconnected-(U1F-GND-PadY24) -> GND
- U1 pad Y9: unconnected-(U1B-GND-PadY9) -> GND

Commit message: fixed missing gnd and vcc nets
Parts:
- removed U30, U31, U32, U33, U34, U35, U36, U37, U38, U39, U40, U41, U42, U43, U44, U45, U46, U47, U48, U49, U50, U51, U52, U53, U54: 74ACT245PC, 16DIP_74ACT:PDIP20_26P42X6P6_ONS
- added J1: Conn_02x08_Top_Bottom, Connector_IDC:IDC-Header_2x08_P2.54mm_Vertical, F.Cu at (122.8, 91.4)
Connections:
- U1 pad AA6: unconnected-(U1C-VCCO_18-PadAA6) -> VCCO
- U1 pad AD7: unconnected-(U1C-VCCO_18-PadAD7) -> VCCO
- U1 pad B13: unconnected-(U1C-VCCO_1-PadB13) -> VCCO
- U1 pad B23: unconnected-(U1C-VCCO_15-PadB23) -> VCCO
- U1 pad C10: unconnected-(U1C-VCCO_16-PadC10) -> VCCO
- U1 pad D17: unconnected-(U1C-VCCO_3-PadD17) -> VCCO
- U1 pad D7: unconnected-(U1A-VCCO_16-PadD7) -> VCCO
- U1 pad E14: unconnected-(U1D-VCCO_1-PadE14) -> VCCO
- U1 pad E24: unconnected-(U1D-VCCO_15-PadE24) -> VCCO
- U1 pad F11: unconnected-(U1D-VCCO_0-PadF11) -> VCCO
- U1 pad F21: unconnected-(U1D-VCCO_15-PadF21) -> VCCO
- U1 pad G18: unconnected-(U1D-VCCO_3-PadG18) -> VCCO
- U1 pad G8: unconnected-(U1A-VCCO_16-PadG8) -> VCCO
- U1 pad H25: unconnected-(U1D-VCCO_11-PadH25) -> VCCO
- U1 pad H5: unconnected-(U1A-VCCO_12-PadH5) -> VCCO
- U1 pad J12: unconnected-(U1D-VCCO_0-PadJ12) -> VCCO
- U1 pad J22: unconnected-(U1D-VCCO_11-PadJ22) -> VCCO
- U1 pad K13: unconnected-(U1D-VCCINT-PadK13) -> VccINT
- U1 pad L6: unconnected-(U1A-VCCO_12-PadL6) -> VCCO
- U1 pad M9: unconnected-(U1B-VCCAUX-PadM9) -> VccAUX
- U1 pad P11: unconnected-(U1E-VCCINT-PadP11) -> VccINT
- U1 pad P7: unconnected-(U1B-VCCO_12-PadP7) -> VCCO
- U1 pad P9: unconnected-(U1B-VCCAUX-PadP9) -> VccAUX
- U1 pad V11: unconnected-(U1F-TCK_0-PadV11) -> TCK
- U1 pad V12: unconnected-(U1F-TDO_0-PadV12) -> TDO
- U1 pad V13: unconnected-(U1F-TDI_0-PadV13) -> TDI
- U1 pad V25: unconnected-(U1F-VCCO_13-PadV25) -> VCCO
- U1 pad W13: unconnected-(U1F-TMS_0-PadW13) -> TMS
Routing:
- net GND: track 0.00 -> 90.5 mm, vias 0 -> 128
- net VccINT: track 0.00 -> 14.1 mm
- net VCCO: track 0.00 -> 2.12 mm, vias 0 -> 3
- net VccAUX: track 0.00 -> 0.71 mm, vias 0 -> 1
- net TMS: track 0.00 -> 0.71 mm, vias 0 -> 1
- net TDO: track 0.00 -> 0.71 mm, vias 0 -> 1
- net TDI: track 0.00 -> 0.71 mm, vias 0 -> 1
- net TCK: track 0.00 -> 0.71 mm, vias 0 -> 1
- added copper zone on B.Cu, net GND
Other:
- copper layers 2 -> 4

Commit message: more work
Routing:
- net VCCO: track 2.12 -> 123.0 mm, vias 3 -> 31
- net VccINT: track 14.1 -> 32.5 mm, vias 0 -> 38
- net VccAUX: track 0.71 -> 9.90 mm, vias 1 -> 12
- added copper zone on In2.Cu, net VccINT

Commit message: vcco layout
Parts:
- moved J1 89.3 mm to (141.5, 178.8)
Routing:
- net VCCO: track 123.0 -> 213.7 mm
- net VccINT: track 32.5 -> 26.9 mm
- net VccAUX: track 9.90 -> 8.49 mm
- net GND: track 90.5 -> 89.8 mm, vias 128 -> 127
- added copper zone on In2.Cu, net VccAUX

Commit message: setup mtttx ports to use case 9
Parts:
- removed C1, C15: 220uF, Capacitor_Tantalum_SMD:CP_EIA-3528-12_Kemet-T
- removed C16, C2: 15nF, Capacitor_Tantalum_SMD:CP_EIA-3528-12_Kemet-T
- removed C17, C3: 1uF, Capacitor_Tantalum_SMD:CP_EIA-3528-12_Kemet-T
- removed C18, C4: 470nF, Capacitor_Tantalum_SMD:CP_EIA-3528-12_Kemet-T
- removed C19, C5: 120pF, Capacitor_Tantalum_SMD:CP_EIA-3528-12_Kemet-T
- removed C20, C6: 470uF, Capacitor_Tantalum_SMD:CP_EIA-3528-12_Kemet-T
- removed L1, L3: 680nH, Inductor_SMD:L_Coilcraft_XAL7050-XXX
- removed Q1, Q2, Q5, Q6: STP40NF03L, Package_TO_SOT_THT:TO-220-3_Vertical
- removed U10, U11, U12, U13, U14, U15, U16, U17, U18, U19, U20, U21, U22, U23, U24, U25, U26, U27, U3, U4, U5, U6, U7, U8, U9: 74ACT245MTC, test_bufferchip_libraryfootprint:TSSOP20_4P4X6P5_ONS
- removed U2, U29: LM3150MHX/NOPB, lm3150Library:MXA14A
- added C21: 470uF, Capacitor_Tantalum_SMD:CP_EIA-3528-12_Kemet-T, F.Cu at (152.1, 163.8)
- added C7: 470uF, Capacitor_Tantalum_SMD:CP_EIA-3528-12_Kemet-T, F.Cu at (169.9, 122.7)
- added J2: Conn_02x20_Counter_Clockwise, Connector_PinHeader_2.54mm:PinHeader_2x20_P2.54mm_Vertical, F.Cu at (202.0, 120.4)
- added J3: Conn_02x20_Counter_Clockwise, Connector_PinHeader_2.54mm:PinHeader_2x20_P2.54mm_Vertical, F.Cu at (110.7, 120.9)
- added J4: Conn_02x20_Counter_Clockwise, Connector_PinHeader_2.54mm:PinHeader_2x20_P2.54mm_Vertical, F.Cu at (117.9, 120.9)
- added J5: Conn_02x20_Counter_Clockwise, Connector_PinHeader_2.54mm:PinHeader_2x20_P2.54mm_Vertical, F.Cu at (125.1, 120.9)
- added J6: Conn_02x20_Counter_Clockwise, Connector_PinHeader_2.54mm:PinHeader_2x20_P2.54mm_Vertical, F.Cu at (210.4, 120.7)
- added J7: Conn_02x20_Counter_Clockwise, Connector_PinHeader_2.54mm:PinHeader_2x20_P2.54mm_Vertical, F.Cu at (217.6, 120.7)
- added X1: SG-5032CCN, Oscillator:Oscillator_SMD_SeikoEpson_SG8002LB-4Pin_5.0x3.2mm, F.Cu at (162.2, 164.6)
- moved C11 60.5 mm to (181.1, 162.6)
- moved C9 46.7 mm to (167.5, 168.4)
- moved C10 45.3 mm to (175.2, 176.5)
- moved C12 40.0 mm to (180.4, 171.2)
- moved Q3 37.1 mm to (167.3, 172.9)
- moved U28 32.3 mm to (174.7, 166.7)
- moved C13 23.1 mm to (183.4, 150.2)
- moved Q4 20.1 mm to (182.6, 167.8)
- moved J1 16.2 mm to (157.0, 173.8), turned to -90 degrees
- moved L2 8.61 mm to (187.8, 156.4)
- moved C14 8.23 mm to (186.2, 172.2)
- moved C8 1.97 mm to (176.2, 125.0)
Connections:
- U1 pad AA3: unconnected-(U1C-MGTAVTTRX_118-PadAA3) -> GND
- U1 pad AC1: unconnected-(U1C-MGTRXN1_118-PadAC1) -> GND
- U1 pad AC16: unconnected-(U1G-IO_L9N_CC_GC_4-PadAC16) -> CLK
- U1 pad AC3: unconnected-(U1C-MGTAVCC_118-PadAC3) -> VccINT
- U1 pad AC4: unconnected-(U1C-MGTAVCC_118-PadAC4) -> VccINT
- U1 pad AD3: unconnected-(U1C-MGTAVCCPLL_118-PadAD3) -> GND
- U1 pad AE3: unconnected-(U1C-MGTAVTTTX_118-PadAE3) -> GND
- U1 pad B3: unconnected-(U1A-MGTAVTTTX_116-PadB3) -> GND
- U1 pad C3: unconnected-(U1A-MGTAVTTRX_116-PadC3) -> GND
- U1 pad E3: unconnected-(U1A-MGTAVCC_116-PadE3) -> VccINT
- U1 pad E4: unconnected-(U1A-MGTAVCC_116-PadE4) -> VccINT
- U1 pad F3: unconnected-(U1A-MGTAVCCPLL_116-PadF3) -> GND
- U1 pad G3: unconnected-(U1A-MGTAVTTTX_116-PadG3) -> GND
- U1 pad H3: unconnected-(U1A-MGTAVTTTX_112-PadH3) -> GND
- U1 pad J3: unconnected-(U1A-MGTAVTTRX_112-PadJ3) -> GND
- U1 pad L9: unconnected-(U1A-GND-PadL9) -> GND
- U1 pad M3: unconnected-(U1B-MGTAVCCPLL_112-PadM3) -> GND
- U1 pad N3: unconnected-(U1B-MGTAVTTTX_112-PadN3) -> GND
- U1 pad P3: unconnected-(U1B-MGTAVTTTX_114-PadP3) -> GND
- U1 pad R18: unconnected-(U1E-VCCINT-PadR18) -> VccINT
- U1 pad R3: unconnected-(U1B-MGTAVTTRX_114-PadR3) -> GND
- U1 pad U3: unconnected-(U1B-MGTAVCC_114-PadU3) -> VccINT
- U1 pad U4: unconnected-(U1B-MGTAVCC_114-PadU4) -> VccINT
- U1 pad V3: unconnected-(U1B-MGTAVCCPLL_114-PadV3) -> GND
- U1 pad W3: unconnected-(U1B-MGTAVTTTX_114-PadW3) -> GND
- U1 pad Y3: unconnected-(U1B-MGTAVTTTX_118-PadY3) -> GND
Routing:
- net VCCO: track 213.7 -> 21.9 mm, vias 31 -> 32
- net GND: track 89.8 -> 101.8 mm, vias 127 -> 144
- net CLK: track 0.00 -> 7.85 mm, vias 0 -> 2
- net unconnected-(U1C-MGTRXP1_118-PadAD1): track 0.00 -> 5.02 mm
- net VccINT: track 26.9 -> 31.1 mm, vias 38 -> 45
- added copper zone on In1.Cu, net VCCO
- added copper zone on In2.Cu, net VCCO
- added copper zone on In1.Cu, net VccINT
Other:
- board text added: "VCCAUX"
- board text added: "VCCINT"
- board text added: "VCCO"

Commit message: more work
Parts:
- removed C10: 15nF, Capacitor_Tantalum_SMD:CP_EIA-3528-12_Kemet-T
- removed C11: 1uF, Capacitor_Tantalum_SMD:CP_EIA-3528-12_Kemet-T
- removed C14, C21: 470uF, Capacitor_Tantalum_SMD:CP_EIA-3528-12_Kemet-T
- removed C9: 220uF, Capacitor_Tantalum_SMD:CP_EIA-3528-12_Kemet-T
- removed J5, J6, J7: Conn_02x20_Counter_Clockwise, Connector_PinHeader_2.54mm:PinHeader_2x20_P2.54mm_Vertical
- removed L2: 680nH, Inductor_SMD:L_Coilcraft_XAL7050-XXX
- removed Q3, Q4: STP40NF03L, Package_TO_SOT_THT:TO-220-3_Vertical
- removed U28: LM3150MHX/NOPB, lm3150Library:MXA14A
- added C1: 470uF, Capacitor_Tantalum_SMD:CP_EIA-3528-12_Kemet-T, B.Cu at (157.7, 130.4)
- added C15: 470uF, Capacitor_Tantalum_SMD:CP_EIA-3528-12_Kemet-T, B.Cu at (174.5, 151.6)
- added C2: 470uF, Capacitor_Tantalum_SMD:CP_EIA-3528-12_Kemet-T, B.Cu at (161.0, 143.3)
- added C3: 470uF, Capacitor_Tantalum_SMD:CP_EIA-3528-12_Kemet-T, B.Cu at (163.4, 130.5)
- added C4: 470uF, Capacitor_Tantalum_SMD:CP_EIA-3528-12_Kemet-T, B.Cu at (174.3, 155.9)
- C12: value 470nF -> 470uF; moved to B.Cu
- C13: value 120pF -> 470uF; moved to B.Cu
- C7, C8, X1: moved to B.Cu
- J1: value Conn_02x08_Top_Bottom -> Conn_02x30_Counter_Clockwise; footprint Connector_IDC:IDC-Header_2x08_P2.54mm_Vertical -> Connector_PinHeader_1.27mm:PinHeader_2x30_P1.27mm_Vertical_SMD
- J2, J3, J4: value Conn_02x20_Counter_Clockwise -> Conn_02x30_Counter_Clockwise; footprint Connector_PinHeader_2.54mm:PinHeader_2x20_P2.54mm_Vertical -> Connector_PinHeader_1.27mm:PinHeader_2x30_P1.27mm_Vertical_SMD
- moved J2 65.0 mm to (140.2, 140.6)
- moved J4 58.7 mm to (157.6, 164.2), turned to -90 degrees
- moved J3 53.4 mm to (164.1, 123.4), turned to -90 degrees
- moved C12 43.0 mm to (154.1, 137.2), turned to 180 degrees
- moved J1 37.0 mm to (181.6, 146.2), turned to 0 degrees
- moved C8 35.9 mm to (156.1, 154.8)
- moved C7 34.0 mm to (147.0, 147.8), turned to 90 degrees
- moved C13 21.2 mm to (170.4, 133.4), turned to 180 degrees
- moved X1 3.86 mm to (161.9, 160.7), turned to 90 degrees
- moved U1 3.75 mm to (161.7, 144.0)
Connections:
- C12 pad 1: Net-(Q3-S) -> VCCO
- C12 pad 2: Net-(U28-BST) -> GND
- C13 pad 1: VccAUX -> VCCO
- C13 pad 2: Net-(U28-FB) -> GND
- C7 pad 1: VccINT -> VccAUX
- J1 pad 1: TDO -> unconnected-(J1-Pin_1-Pad1)
- J1 pad 2: TDI -> unconnected-(J1-Pin_2-Pad2)
- J1 pad 4: TCK -> unconnected-(J1-Pin_4-Pad4)
- J1 pad 5: TMS -> unconnected-(J1-Pin_5-Pad5)
- U1 pad P4: unconnected-(U1B-MGTRREF_112-PadP4) -> GND
- U1 pad P5: unconnected-(U1B-MGTAVTTRXC-PadP5) -> GND
Routing:
- net VCCO: track 21.9 -> 31.8 mm, vias 32 -> 31
- net CLK: track 7.85 -> 5.30 mm
- net GND: track 101.8 -> 102.5 mm, vias 144 -> 145
- net VccINT: vias 45 -> 46
- added copper zone on B.Cu, net CLK
- added copper zone on B.Cu, net VCCO
- added copper zone on B.Cu, net VccAUX
- removed copper zone on B.Cu, net GND
