File: XC5VLX30T_testboard/XC5VLX30T_testboard.kicad_sch (KiCad schematic)
At the start: 1 part, among them U1 XC5VLX30T-1FFG665I

Commit message: h
Parts:
- removed U1: XC5VLX30T-1FFG665I, 665-FBGA_XIL, symbol 2024-06-14_00-02-59:XC5VLX30T-1FFG665I
- added C1, C15, C9: 220uF, Capacitor_Tantalum_SMD:CP_EIA-3528-12_Kemet-T, symbol Device:C
- added C10, C16, C2: 15nF, Capacitor_Tantalum_SMD:CP_EIA-3528-12_Kemet-T, symbol Device:C
- added C11, C17, C3: 1uF, Capacitor_Tantalum_SMD:CP_EIA-3528-12_Kemet-T, symbol Device:C
- added C12, C18, C4: 470nF, Capacitor_Tantalum_SMD:CP_EIA-3528-12_Kemet-T, symbol Device:C
- added C13, C19, C5: 120pF, Capacitor_Tantalum_SMD:CP_EIA-3528-12_Kemet-T, symbol Device:C
- added C14, C20, C6, C8: 470uF, Capacitor_Tantalum_SMD:CP_EIA-3528-12_Kemet-T, symbol Device:C
- added L1, L2, L3: 680nH, Inductor_SMD:L_Coilcraft_XAL7050-XXX, symbol Device:L
- added Q1, Q2, Q3, Q4, Q5, Q6: STP40NF03L, Package_TO_SOT_THT:TO-220-3_Vertical, symbol Transistor_FET:IRF3205
- added R1, R5, R9: 5.9k, symbol Device:R_US
- added R10, R2, R6: 1.1k, symbol Device:R_US
- added R11, R3, R7: 6.65k, symbol Device:R_US
- added R12, R4, R8: 10k, symbol Device:R_US
- added U1: XC5VLX30T-1FFG665C, Library:digikey665-FBGA_XIL, symbol digikeyvirtex:XC5VLX30T-1FFG665C
- added U10, U11, U12, U13, U14, U15, U16, U17, U18, U19, U20, U21, U22, U23, U24, U25, U26, U27, U3, U4, U5, U6, U7, U8, U9: 74ACT245MTC, TSSOP20_4P4X6P5_ONS, symbol BUFFERCHIPPY:74ACT245MTC
- added U2, U28, U29: LM3150MHX/NOPB, lm3150Library:MXA14A, symbol LM3150:LM3150MHX_NOPB
- added U30, U31, U32, U33, U34, U35, U36, U37, U38, U39, U40, U41, U42, U43, U44, U45, U46, U47, U48, U49, U50, U51, U52, U53, U54: 74ACT245PC, 16DIP_74ACT:PDIP20_26P42X6P6_ONS, symbol 74ACT_16DIP:74ACT245PC
Connections:
- new net: C9.1, Q3.2 (D), R5.1, U28.2 (VIN)
- new net: C13.2, R7.2, R8.1, U28.4 (FB)
- new net: C11.1, U28.1 (VCC)
- new net: C18.1, L3.2, Q5.3 (S), Q6.2 (D), R10.1, U29.10 (SW)
- new net: C3.1, U2.1 (VCC)
- new net: C4.1, L1.2, Q1.3 (S), Q2.2 (D), R2.1, U2.10 (SW)
- new net: Q1.1 (G), U2.11 (HG)
- new net: C4.2, U2.12 (BST)
- new net: Q2.1 (G), U2.13 (LG)
- new net: C1.1, Q1.2 (D), R1.1, U2.2 (VIN)
- new net: C5.2, R3.2, R4.1, U2.4 (FB)
- new net: C2.1, U2.6 (SS)
- new net: R1.2, U2.7 (RON)
- new net: R2.2, U2.8 (ILIM)
- new net: C15.1, Q5.2 (D), R9.1, U29.2 (VIN)
- new net: R9.2, U29.7 (RON)
- new net: Q3.1 (G), U28.11 (HG)
- new net: C12.1, L2.2, Q3.3 (S), Q4.2 (D), R6.1, U28.10 (SW)
- new net: R6.2, U28.8 (ILIM)
- new net: R5.2, U28.7 (RON)
- new net: C17.1, U29.1 (VCC)
- new net: C19.2, R11.2, R12.1, U29.4 (FB)
- new net: C10.1, U28.6 (SS)
- new net: Q4.1 (G), U28.13 (LG)
- new net: C12.2, U28.12 (BST)
- new net: R10.2, U29.8 (ILIM)
- new net: Q5.1 (G), U29.11 (HG)
- new net: C18.2, U29.12 (BST)
- new net: Q6.1 (G), U29.13 (LG)
- new net: C16.1, U29.6 (SS)
- new net GND: C1.2, C10.2, C11.2, C14.2, C15.2, C16.2, C17.2, C2.2, C20.2, C3.2, C6.2, C8.2, C9.2, Q2.3 (S), Q4.3 (S), Q6.3 (S), R12.2, R4.2, R8.2, U1.A11 (GND), U1.A16 (GND), U1.A2 (GND), U1.A21 (GND), U1.A26 (GND), U1.A6 (GND), U1.AA11 (GND), U1.AA21 (GND), U1.AA26 (GND), U1.AA4 (GND), U1.AB18 (GND), U1.AB2 (GND), U1.AB8 (GND), U1.AC15 (GND), U1.AC2 (GND), U1.AC25 (GND), U1.AC5 (GND), U1.AD12 (GND), U1.AD22 (GND), U1.AE19 (GND), U1.AE4 (GND), U1.AE9 (GND), U1.AF11 (GND), U1.AF16 (GND), U1.AF2 (GND), U1.AF21 (GND), U1.AF26 (GND), U1.AF6 (GND), U1.B18 (GND), U1.B8 (GND), U1.C15 (GND), U1.C20 (GND), U1.C25 (GND), U1.C4 (GND), U1.C5 (GND), U1.D12 (GND), U1.D2 (GND), U1.D22 (GND), U1.E19 (GND), U1.E2 (GND), U1.E9 (GND), U1.F16 (GND), U1.F26 (GND), U1.F4 (GND), U1.F6 (GND), U1.G13 (GND), U1.G23 (GND), U1.H10 (GND), U1.H14 (GND), U1.H16 (GND), U1.H20 (GND), U1.J13 (GND), U1.J15 (GND), U1.J17 (GND), U1.J4 (GND), U1.J7 (GND), U1.K10 (GND), U1.K12 (GND), U1.K14 (GND), U1.K16 (GND), U1.K18 (GND), U1.K2 (GND), U1.K24 (GND), U1.L11 (GND), U1.L13 (GND), U1.L15 (GND), U1.L17 (GND), U1.L19 (GND), U1.L2 (GND), U1.L21 (GND), U1.L26 (GND), U1.M10 (GND), U1.M12 (GND), U1.M16 (GND), U1.M18 (GND), U1.M4 (GND), U1.M8 (GND), U1.N11 (GND), U1.N13 (GND), U1.N17 (GND), U1.N19 (GND), U1.N25 (GND), U1.N5 (GND), U1.N9 (GND), U1.P10 (GND), U1.P12 (GND), U1.P16 (GND), U1.P18 (GND), U1.P22 (GND), U1.R11 (GND), U1.R13 (GND), U1.R17 (GND), U1.R19 (GND), U1.R4 (GND), U1.R9 (GND), U1.T10 (GND), U1.T12 (GND), U1.T14 (GND), U1.T16 (GND), U1.T18 (GND), U1.T2 (GND), U1.T21 (GND), U1.T26 (GND), U1.T6 (GND), U1.U11 (GND), U1.U13 (GND), U1.U15 (GND), U1.U17 (GND), U1.U19 (GND), U1.U2 (GND), U1.U23 (GND), U1.U9 (GND), U1.V10 (GND), U1.V14 (GND), U1.V16 (GND), U1.V18 (GND), U1.V20 (GND), U1.V4 (GND), U1.V5 (GND), U1.W12 (GND), U1.W15 (GND), U1.W17 (GND), U1.W19 (GND), U1.W7 (GND), U1.Y14 (GND), U1.Y24 (GND), U1.Y9 (GND), U2.14 (PGND), U2.5 (SGND), U2.9 (SGND), U28.14 (PGND), U28.5 (SGND), U28.9 (SGND), U29.14 (PGND), U29.5 (SGND), U29.9 (SGND)
- new net VCCO: C19.1, C20.1, C8.1, L3.1, R11.1, U1.AA16 (VCCO_2), U1.AB13 (VCCO_4), U1.AB23 (VCCO_17), U1.AC10 (VCCO_18), U1.AC20 (VCCO_17), U1.AD17 (VCCO_2), U1.AE14 (VCCO_4), U1.AE24 (VCCO_17), U1.M23 (VCCO_11), U1.R24 (VCCO_13), U1.W22 (VCCO_13)
- new net VccAUX: C13.1, C14.1, L2.1, R7.1, U1.K9 (VCCAUX), U1.M19 (VCCAUX), U1.N20 (VCCAUX), U1.P19 (VCCAUX), U1.T19 (VCCAUX), U1.T9 (VCCAUX), U1.U8 (VCCAUX), U1.V19 (VCCAUX), U1.W10 (VCCAUX), U1.Y19 (VCCAUX)
- new net VccINT: C5.1, C6.1, L1.1, R3.1, U1.H15 (VCCINT), U1.H17 (VCCINT), U1.J14 (VCCINT), U1.J16 (VCCINT), U1.J18 (VCCINT), U1.K15 (VCCINT), U1.K17 (VCCINT), U1.K19 (VCCINT), U1.L10 (VCCINT), U1.L12 (VCCINT), U1.L14 (VCCINT), U1.L16 (VCCINT), U1.L18 (VCCINT), U1.M11 (VCCINT), U1.M13 (VCCINT), U1.M17 (VCCINT), U1.N10 (VCCINT), U1.N12 (VCCINT), U1.N16 (VCCINT), U1.N18 (VCCINT), U1.P13 (VCCINT), U1.P17 (VCCINT), U1.R10 (VCCINT), U1.R12 (VCCINT), U1.R16 (VCCINT), U1.T11 (VCCINT), U1.T13 (VCCINT), U1.T15 (VCCINT), U1.T17 (VCCINT), U1.U10 (VCCINT), U1.U14 (VCCINT), U1.U16 (VCCINT), U1.U18 (VCCINT), U1.V15 (VCCINT), U1.V17 (VCCINT), U1.W18 (VCCINT)
- no-connect marks 0 -> 6

Commit message: fixed missing gnd and vcc nets
Parts:
- removed U30, U31, U32, U33, U34, U35, U36, U37, U38, U39, U40, U41, U42, U43, U44, U45, U46, U47, U48, U49, U50, U51, U52, U53, U54: 74ACT245PC, 16DIP_74ACT:PDIP20_26P42X6P6_ONS, symbol 74ACT_16DIP:74ACT245PC
- added J1: Conn_02x08_Top_Bottom, Connector_IDC:IDC-Header_2x08_P2.54mm_Vertical, symbol Connector_Generic:Conn_02x08_Top_Bottom
Connections:
- net VCCO: now also U1.AA6 (VCCO_18), U1.AD7 (VCCO_18), U1.B13 (VCCO_1), U1.B23 (VCCO_15), U1.C10 (VCCO_16), U1.D17 (VCCO_3), U1.D7 (VCCO_16), U1.E14 (VCCO_1), U1.E24 (VCCO_15), U1.F11 (VCCO_0), U1.F21 (VCCO_15), U1.G18 (VCCO_3), U1.G8 (VCCO_16), U1.H25 (VCCO_11), U1.H5 (VCCO_12), U1.J12 (VCCO_0), U1.J22 (VCCO_11), U1.L6 (VCCO_12), U1.P7 (VCCO_12), U1.V25 (VCCO_13)
- net VccAUX: now also U1.M9 (VCCAUX), U1.P9 (VCCAUX)
- net VccINT: now also U1.K13 (VCCINT), U1.P11 (VCCINT)
- net TCK: now reaches U1.V11 (TCK_0)
- net TCK: now also J1.4 (Pin_4)
- net TDO: now reaches U1.V12 (TDO_0)
- net TDO: now also J1.1 (Pin_1)
- net TDI: now reaches U1.V13 (TDI_0)
- net TDI: now also J1.2 (Pin_2)
- net TMS: now reaches U1.W13 (TMS_0)
- net TMS: now also J1.5 (Pin_5)

Commit message: more work
Parts:
- removed C1, C15: 220uF, Capacitor_Tantalum_SMD:CP_EIA-3528-12_Kemet-T, symbol Device:C
- removed C16, C2: 15nF, Capacitor_Tantalum_SMD:CP_EIA-3528-12_Kemet-T, symbol Device:C
- removed C17, C3: 1uF, Capacitor_Tantalum_SMD:CP_EIA-3528-12_Kemet-T, symbol Device:C
- removed C18, C4: 470nF, Capacitor_Tantalum_SMD:CP_EIA-3528-12_Kemet-T, symbol Device:C
- removed C19, C5: 120pF, Capacitor_Tantalum_SMD:CP_EIA-3528-12_Kemet-T, symbol Device:C
- removed C20, C6: 470uF, Capacitor_Tantalum_SMD:CP_EIA-3528-12_Kemet-T, symbol Device:C
- removed L1, L3: 680nH, Inductor_SMD:L_Coilcraft_XAL7050-XXX, symbol Device:L
- removed Q1, Q2, Q5, Q6: STP40NF03L, Package_TO_SOT_THT:TO-220-3_Vertical, symbol Transistor_FET:IRF3205
- removed R1, R9: 5.9k, symbol Device:R_US
- removed R10, R2: 1.1k, symbol Device:R_US
- removed R11, R3: 6.65k, symbol Device:R_US
- removed R12, R4: 10k, symbol Device:R_US
- removed U10, U11, U12, U13, U14, U15, U16, U17, U18, U19, U20, U21, U22, U23, U24, U25, U26, U27, U3, U4, U5, U6, U7, U8, U9: 74ACT245MTC, TSSOP20_4P4X6P5_ONS, symbol BUFFERCHIPPY:74ACT245MTC
- removed U2, U29: LM3150MHX/NOPB, lm3150Library:MXA14A, symbol LM3150:LM3150MHX_NOPB
- added C21, C7: 470uF, Capacitor_Tantalum_SMD:CP_EIA-3528-12_Kemet-T, symbol Device:C
Connections:
- net GND: now also U1.L9 (GND), C21.2, C7.2
- net VccAUX: now also C21.1
- net VccINT: now also C7.1
- no-connect marks 6 -> 2

Commit message: setup mtttx ports to use case 9
Parts:
- added J2, J3, J4, J5, J6, J7: Conn_02x20_Counter_Clockwise, Connector_PinHeader_2.54mm:PinHeader_2x20_P2.54mm_Vertical, symbol Connector_Generic:Conn_02x20_Counter_Clockwise
- added X1: SG-5032CCN, Oscillator:Oscillator_SMD_SeikoEpson_SG8002LB-4Pin_5.0x3.2mm, symbol Oscillator:SG-5032CCN
Connections:
- net GND: now also U1.AA3 (MGTAVTTRX_118), U1.AC1 (MGTRXN1_118), U1.AD3 (MGTAVCCPLL_118), U1.AE3 (MGTAVTTTX_118), U1.B3 (MGTAVTTTX_116), U1.C3 (MGTAVTTRX_116), U1.F3 (MGTAVCCPLL_116), U1.G3 (MGTAVTTTX_116), U1.H3 (MGTAVTTTX_112), U1.J3 (MGTAVTTRX_112), U1.M3 (MGTAVCCPLL_112), U1.N3 (MGTAVTTTX_112), U1.P3 (MGTAVTTTX_114), U1.R3 (MGTAVTTRX_114), U1.V3 (MGTAVCCPLL_114), U1.W3 (MGTAVTTTX_114), U1.Y3 (MGTAVTTTX_118), X1.2 (GND)
- net VCCO: now also X1.1 (OE), X1.4 (Vcc)
- net VccINT: now also U1.AC3 (MGTAVCC_118), U1.AC4 (MGTAVCC_118), U1.E3 (MGTAVCC_116), U1.E4 (MGTAVCC_116), U1.R18 (VCCINT), U1.U3 (MGTAVCC_114), U1.U4 (MGTAVCC_114)
- net CLK: now reaches U1.AC16 (IO_L9N_CC_GC_4)
- net CLK: now also X1.3 (OUT)

Commit message: more work
Parts:
- removed C10: 15nF, Capacitor_Tantalum_SMD:CP_EIA-3528-12_Kemet-T, symbol Device:C
- removed C11: 1uF, Capacitor_Tantalum_SMD:CP_EIA-3528-12_Kemet-T, symbol Device:C
- removed C14, C21: 470uF, Capacitor_Tantalum_SMD:CP_EIA-3528-12_Kemet-T, symbol Device:C
- removed C9: 220uF, Capacitor_Tantalum_SMD:CP_EIA-3528-12_Kemet-T, symbol Device:C
- removed J1: Conn_02x08_Top_Bottom, Connector_IDC:IDC-Header_2x08_P2.54mm_Vertical, symbol Connector_Generic:Conn_02x08_Top_Bottom
- removed J2, J3, J4, J5, J6, J7: Conn_02x20_Counter_Clockwise, Connector_PinHeader_2.54mm:PinHeader_2x20_P2.54mm_Vertical, symbol Connector_Generic:Conn_02x20_Counter_Clockwise
- removed L2: 680nH, Inductor_SMD:L_Coilcraft_XAL7050-XXX, symbol Device:L
- removed Q3, Q4: STP40NF03L, Package_TO_SOT_THT:TO-220-3_Vertical, symbol Transistor_FET:IRF3205
- removed R5: 5.9k, symbol Device:R_US
- removed R6: 1.1k, symbol Device:R_US
- removed R7: 6.65k, symbol Device:R_US
- removed R8: 10k, symbol Device:R_US
- removed U28: LM3150MHX/NOPB, lm3150Library:MXA14A, symbol LM3150:LM3150MHX_NOPB
- added C1, C15, C2, C3, C4: 470uF, Capacitor_Tantalum_SMD:CP_EIA-3528-12_Kemet-T, symbol Device:C
- added J1, J2, J3, J4: Conn_02x30_Counter_Clockwise, Connector_PinHeader_1.27mm:PinHeader_2x30_P1.27mm_Vertical_SMD, symbol Connector_Generic:Conn_02x30_Counter_Clockwise
- C12: value 470nF -> 470uF
- C13: value 120pF -> 470uF
Connections:
- net GND: now also C12.2, C13.2, U1.P4 (MGTRREF_112), U1.P5 (MGTAVTTRXC), C1.2, C15.2, C2.2, C3.2, C4.2
- net VCCO: now also C12.1, C13.1, C4.1
- net VccAUX: now also C7.1, C15.1; no longer C13.1
- net VccINT: now also C1.1, C2.1, C3.1; no longer C7.1
- no-connect marks 2 -> 0
Other:
- moved on the sheet: C8, X1

Commit message: routing
routed 240 pins on 4 layer
Connections:
- net GND: now also U1.F2 (MGTTXN1_116); no longer U1.AC1 (MGTRXN1_118), U1.P5 (MGTAVTTRXC)
- net VccINT: now also U1.L3 (MGTAVCC_112), U1.L4 (MGTAVCC_112)
- net IO_L4N_VREF_18: now reaches U1.AE10 (IO_L4N_VREF_18)
- net IO_L2P_18: now reaches U1.AE11 (IO_L2P_18)
- net IO_L0N_18: now reaches U1.AE12 (IO_L0N_18)
- net IO_L18N_17: now reaches U1.AE13 (IO_L18N_17)
- net IO_L16N_17: now reaches U1.AE15 (IO_L16N_17)
- net IO_L15P_17: now reaches U1.AE16 (IO_L15P_17)
- net IO_L14P_17: now reaches U1.AE17 (IO_L14P_17)
- net IO_L13P_17: now reaches U1.AE18 (IO_L13P_17)
- net IO_L9N_CC_17: now reaches U1.AE20 (IO_L9N_CC_17)
- net IO_L8N_CC_17: now reaches U1.AE21 (IO_L8N_CC_17)
- net IO_L5P_17: now reaches U1.AE22 (IO_L5P_17)
- net IO_L4N_VREF_17: now reaches U1.AE23 (IO_L4N_VREF_17)
- net IO_L2P_17: now reaches U1.AE25 (IO_L2P_17)
- net IO_L2N_17: now reaches U1.AE26 (IO_L2N_17)
- net IO_L6N_18: now reaches U1.AF10 (IO_L6N_18)
- net IO_L0P_18: now reaches U1.AF12 (IO_L0P_18)
- net IO_L0P_17: now reaches U1.AF13 (IO_L18P_17)
- net IO_L17N_17: now reaches U1.AF14 (IO_L17N_17)
- net IO_L17P_17: now reaches U1.AF15 (IO_L17P_17)
- net IO_L14N_VREF_17: now reaches U1.AF17 (IO_L14N_VREF_17)
- net IO_L12N_VRP_17: now reaches U1.AF18 (IO_L12N_VRP_17)
- net IO_L12P_VRN_17: now reaches U1.AF19 (IO_L12P_VRN_17)
- net IO_L9P_CC_17: now reaches U1.AF20 (IO_L9P_CC_17)
- net IO_L8P_CC_17: now reaches U1.AF22 (IO_L8P_CC_17)
- net IO_L4P_17: now reaches U1.AF23 (IO_L4P_17)
- net IO_L3N_17: now reaches U1.AF24 (IO_L3N_17)
- net IO_L3P_17: now reaches U1.AF25 (IO_L3P_17)
- net IO_L14P_18: now reaches U1.AE5 (IO_L14P_18)
- net IO_L13P_18: now reaches U1.AE6 (IO_L13P_18)
- net IO_L11N_CC_18: now reaches U1.AE7 (IO_L11N_CC_18)
- net IO_L11P_CC_18: now reaches U1.AE8 (IO_L11P_CC_18)
- net IO_L15N_18: now reaches U1.AF3 (IO_L15N_18)
- net IO_L15P_18: now reaches U1.AF4 (IO_L15P_18)
- net IO_L13N_18: now reaches U1.AF5 (IO_L13N_18)
- net IO_L8P_CC_18: now reaches U1.AF7 (IO_L8P_CC_18)
- net IO_L8N_CC_18: now reaches U1.AF8 (IO_L8N_CC_18)
- net IO_L6P_18: now reaches U1.AF9 (IO_L6P_18)
- no-connect marks 0 -> 25
Other:
- note added: "top layer, 1st bottom row - AF"
- note added: "top layer, 2nd bottom row - AE"

Commit message: plumbing
Parts:
- removed J1, J2, J3, J4: Conn_02x30_Counter_Clockwise, Connector_PinHeader_1.27mm:PinHeader_2x30_P1.27mm_Vertical_SMD, symbol Connector_Generic:Conn_02x30_Counter_Clockwise
- added J1, J2, J3, J4, J5, J6, J7, J8: Conn_01x35_Pin, Connector_PinHeader_1.27mm:PinHeader_1x35_P1.27mm_Vertical, symbol Connector:Conn_01x35_Pin
Connections:
- net IO_L14N_VREF_11: now reaches U1.L25 (IO_L14N_VREF_11)
- net IO_L14P_16: now reaches U1.A4 (IO_L14P_16)
- net IO_L14P_16: now also J3.5 (Pin_5), J3.6 (Pin_6)
- net IO_L16P_16: now reaches U1.B4 (IO_L16P_16)
- net IO_L7P_16: now reaches U1.E6 (IO_L7P_16)
- new net J5PIN1: J3.2 (Pin_2), J3.3 (Pin_3), J3.4 (Pin_4), J5.1 (Pin_1)
Other:
- moved on the sheet: C12, C13, C4, C7, C8

Commit message: fixed missing pins
MGTRXP/MGTRXN wasnt connected to GND
Connections:
- net GND: now also U1.AA1 (MGTRXP0_118), U1.AB1 (MGTRXN0_118), U1.AC1 (MGTRXN1_118), U1.AD1 (MGTRXP1_118), U1.C1 (MGTRXP0_116), U1.D1 (MGTRXN0_116), U1.E1 (MGTRXN1_116), U1.F1 (MGTRXP1_116), U1.J1 (MGTRXP0_112), U1.K1 (MGTRXN0_112), U1.L1 (MGTRXN1_112), U1.M1 (MGTRXP1_112), U1.R1 (MGTRXP0_114), U1.T1 (MGTRXN0_114), U1.U1 (MGTRXN1_114), U1.V1 (MGTRXP1_114)
- no-connect marks 25 -> 24
