File: XC5VLX30T_testboard/XC5VLX30T_testboard.kicad_sch (KiCad schematic)
At the start: 19 parts, among them J1 Conn_01x35_Pin, J2 Conn_01x35_Pin, J3 Conn_01x35_Pin, J4 Conn_01x35_Pin, J5 Conn_01x35_Pin, J6 Conn_01x35_Pin, J7 Conn_01x35_Pin, J8 Conn_01x35_Pin, U1 XC5VLX30T-1FFG665C, X1 SG-5032CCN

Commit message: more routing
Connections:
- net GND: now also J1.1 (Pin_1), J1.14 (Pin_14), J1.21 (Pin_21), J1.28 (Pin_28), J1.35 (Pin_35), J1.7 (Pin_7), J2.1 (Pin_1), J2.14 (Pin_14), J2.21 (Pin_21), J2.28 (Pin_28), J2.35 (Pin_35), J2.7 (Pin_7), J3.1 (Pin_1), J3.14 (Pin_14), J3.21 (Pin_21), J3.28 (Pin_28), J3.35 (Pin_35), J3.7 (Pin_7), J4.1 (Pin_1), J4.14 (Pin_14), J4.21 (Pin_21), J4.28 (Pin_28), J4.35 (Pin_35), J4.7 (Pin_7), J5.1 (Pin_1), J5.14 (Pin_14), J5.21 (Pin_21), J5.28 (Pin_28), J5.35 (Pin_35), J5.7 (Pin_7), J6.1 (Pin_1), J6.14 (Pin_14), J6.21 (Pin_21), J6.28 (Pin_28), J6.35 (Pin_35), J6.7 (Pin_7), J7.1 (Pin_1), J7.14 (Pin_14), J7.21 (Pin_21), J7.28 (Pin_28), J7.35 (Pin_35), J7.7 (Pin_7), J8.1 (Pin_1), J8.14 (Pin_14), J8.21 (Pin_21), J8.28 (Pin_28), J8.35 (Pin_35), J8.7 (Pin_7)
- net IO_L0P_17: now also U1.AC26 (IO_L0P_17)
- net IO_L16P_16: now also J3.4 (Pin_4)
- net IO_L7P_16: now also J3.2 (Pin_2), U1.F5 (IO_L3N_12)
- net IO_L13N_16: now reaches U1.A10 (IO_L13N_16)
- net IO_L15N_16: now reaches U1.A12 (IO_L15N_16)
- net IO_L1N_15: now reaches U1.A13 (IO_L1N_15)
- net IO_L2P_15: now reaches U1.A14 (IO_L2P_15)
- net IO_L2N_15: now reaches U1.A15 (IO_L2N_15)
- net IO_L5N_15: now reaches U1.A17 (IO_L5N_15)
- net IO_L6P_15: now reaches U1.A18 (IO_L6P_15)
- net IO_L6N_15: now reaches U1.A19 (IO_L6N_15)
- net IO_L8P_CC_15: now reaches U1.A20 (IO_L8P_CC_15)
- net IO_L13N_15: now reaches U1.A22 (IO_L13N_15)
- net IO_L14P_15: now reaches U1.A23 (IO_L14P_15)
- net IO_L14N_VREF_15: now reaches U1.A24 (IO_L14N_VREF_15)
- net IO_L17N_15: now reaches U1.A25 (IO_L17N_15)
- net IO_L17P_12: now reaches U1.M6 (IO_L17P_12)
- net IO_L13_N_12: now reaches U1.R5 (IO_L13N_12)
- net IO_L15_N_12: now reaches U1.R6 (IO_L15P_12)
- net IO_L19_N_12: now reaches U1.R7 (IO_L19N_12)
- net IO_L13P_12: now reaches U1.T5 (IO_L13P_12)
- net IO_L15N_12: now reaches U1.T7 (IO_L15N_12)
- net IO_L11N_CC_12: now reaches U1.U5 (IO_L11N_CC_12)
- net IO_L6P_12: now reaches U1.V6 (IO_L6P_12)
- net IO_L2N_12: now reaches U1.W4 (IO_L2N_12)
- net IO_L4P_12: now reaches U1.W5 (IO_L4P_12)
- net IO_L4N_VREF_12: now reaches U1.W6 (IO_L4N_VREF_12)
- net IO_L2P_12: now reaches U1.Y4 (IO_L2P_12)
- net IO_L0N_12: now reaches U1.Y5 (IO_L0N_12)
- net IO_L0P_12: now reaches U1.Y6 (IO_L0P_12)
- net IO_L6N_D6_2: now reaches U1.AA14 (IO_L6N_D6_2)
- net IO_L1N_SM7N_13: now reaches U1.R25 (IO_L1N_SM7N_13)
- net IO_L0N_SM8N_13: now reaches U1.R26 (IO_L0N_SM8N_13)
- net IO_L6P_SM3P_13: now reaches U1.T24 (IO_L6P_SM3P_13)
- net IO_L5N_SM4N_13: now reaches U1.T25 (IO_L5N_SM4N_13)
- net IO_L5P_SM4P_13: now reaches U1.U25 (IO_L5P_SM4P_13)
- net IO_L4P_13: now reaches U1.U26 (IO_L4P_13)
- net IO_L7N_SM2N_13: now reaches U1.V24 (IO_L7N_SM2N_13)
- net IO_L4N_VREF_13: now reaches U1.V26 (IO_L4N_VREF_13)
- net IO_L11N_CC_13: now reaches U1.W23 (IO_L11N_CC_13)
- net IO_L9P_CC_SM0P_13: now reaches U1.W24 (IO_L9P_CC_SM0P_13)
- net IO_L8N_CC_SM1N_13: now reaches U1.W25 (IO_L8N_CC_SM1N_13)
- net IO_L8P_CC_SM1P_13: now reaches U1.W26 (IO_L8P_CC_SM1P_13)
- net IO_L12N_VRP_13: now reaches U1.Y25 (IO_L12N_VRP_13)
- net IO_L12P_VRN_13: now reaches U1.Y26 (IO_L12P_VRN_13)
- net IO_L9P_CC_11: now reaches U1.K22 (IO_L9P_CC_11)
- net IO_L9N_CC_11: now reaches U1.K23 (IO_L9N_CC_11)
- net IO_L15N_SM13N_11: now reaches U1.K25 (IO_L15N_SM13N_11)
- net IO_L14P_11: now reaches U1.K26 (IO_L14P_11)
- net IO_L10N_CC_SM15N_11: now reaches U1.L22 (IO_L10N_CC_SM15N_11)
- net IO_L10P_CC_SM15P_11: now reaches U1.L23 (IO_L10P_CC_SM15P_11)
- net IO_L15P_CC_SM13P_11: now reaches U1.L24 (IO_L15P_SM13P_11)
- net IO_L19N_SM9N_11: now reaches U1.M22 (IO_L19N_SM9N_11)
- net IO_L17N_SM11N_11: now reaches U1.M24 (IO_L17N_SM11N_11)
- net IO_L17P_SM11P_11: now reaches U1.M25 (IO_L17P_SM11P_11)
- net IO_L16N_SM12N_11: now reaches U1.M26 (IO_L16N_SM12N_11)
- net IO_L19P_SM9P_11: now reaches U1.N22 (IO_L19P_SM9P_11)
- net IO_L18N_SM10N_11: now reaches U1.N23 (IO_L18N_SM10N_11)
- net IO_L18P_SM10P_11: now reaches U1.N24 (IO_L18P_SM10P_11)
- net IO_L2N_SM6N_13: now reaches U1.P23 (IO_L2N_SM6N_13)
- net IO_L2P_SM6P_13: now reaches U1.P24 (IO_L2P_SM6P_13)
- net IO_L1P_SM7P_13: now reaches U1.P25 (IO_L1P_SM7P_13)
- net IO_L0P_SM8P_13: now reaches U1.P26 (IO_L0P_SM8P_13)
- net IO_L3N_SM5N_13: now reaches U1.R22 (IO_L3N_SM5N_13)
- net IO_L3P_SM5P_13: now reaches U1.R23 (IO_L3P_SM5P_13)
- net IO_L10P_CC_15: now reaches U1.D21 (IO_L10P_CC_15)
- net IO_L12P_VRN_15: now reaches U1.D23 (IO_L12P_VRN_15)
- net IO_L16N_15: now reaches U1.D24 (IO_L16P_15)
- net IO_L16N_15: now also U1.C24 (IO_L16N_15)
- net IO_L19N_15: now reaches U1.D25 (IO_L19N_15)
- net IO_L19P_15: now reaches U1.D26 (IO_L19P_15)
- net IO_L4P_11: now reaches U1.E23 (IO_L4P_11)
- net IO_L0N_11: now reaches U1.E25 (IO_L0N_11)
- net IO_L0P_11: now reaches U1.E26 (IO_L0P_11)
- net IO_L3P_11: now reaches U1.F24 (IO_L3P_11)
- net IO_L1P_11: now reaches U1.F25 (IO_L1P_11)
- net IO_L6P_11: now reaches U1.G22 (IO_L6P_11)
- net IO_L3N_11: now reaches U1.G24 (IO_L3N_11)
- net IO_L2N_11: now reaches U1.G25 (IO_L2N_11)
- net IO_L1N_11: now reaches U1.G26 (IO_L1N_11)
- net IO_L6N_11: now reaches U1.H22 (IO_L6N_11)
- net IO_L7N_11: now reaches U1.J23 (IO_L7N_11)
- net IO_L12N_VRP_11: now reaches U1.J24 (IO_L12N_VRP_11)
- net IO_L13P_11: now reaches U1.J25 (IO_L13P_11)
- net IO_L13N_11: now reaches U1.J26 (IO_L13N_11)
- net IO_L14N_VREF_13: now reaches U1.AA24 (IO_L14N_VREF_13)
- net IO_L13P_13: now reaches U1.AA25 (IO_L13P_13)
- net IO_L7P_GC_VRN_4: now reaches U1.AB14 (IO_L7P_GC_VRN_4)
- net IO_L15P_13: now reaches U1.AB24 (IO_L15P_13)
- net IO_L14P_13: now reaches U1.AB25 (IO_L14P_13)
- net IO_L13N_13: now reaches U1.AB26 (IO_L13N_13)
- net IO_L3P_GC_D9_4: now reaches U1.AC11 (IO_L3P_GC_D9_4)
- net IO_L5P_GC_4: now reaches U1.AC12 (IO_L5P_GC_4)
- net IO_L5N_GC_4: now reaches U1.AC13 (IO_L5N_GC_4)
- net IO_L7N_GC_VRP: now reaches U1.AC14 (IO_L7N_GC_VRP_4)
- net IO_L8P_CC_GC_4: now reaches U1.AC17 (IO_L8P_CC_GC_4)
- net IO_L6P_GC_4: now reaches U1.AC18 (IO_L6P_GC_4)
- net IO_L4N_GC_VREF_4: now reaches U1.AC19 (IO_L4N_GC_VREF_4)
- net IO_L11P_CC_17: now reaches U1.AC21 (IO_L11P_CC_17)
- net IO_L7P_17: now reaches U1.AC22 (IO_L7P_17)
- net IO_L6N_17: now reaches U1.AC23 (IO_L6N_17)
- net IO_L6P_17: now reaches U1.AC24 (IO_L6P_17)
- net IO_L4P_18: now reaches U1.AD10 (IO_L4P_18)
- net IO_L2N_18: now reaches U1.AD11 (IO_L2N_18)
- net IO_L19P_17: now reaches U1.AD13 (IO_L19P_17)
- net IO_L19N_17: now reaches U1.AD14 (IO_L19N_17)
- net IO_L16P_17: now reaches U1.AD15 (IO_L16P_17)
- net IO_L15N_17: now reaches U1.AD16 (IO_L15N_17)
- net IO_L13N_17: now reaches U1.AD18 (IO_L13N_17)
- net IO_L10P_CC_17: now reaches U1.AD19 (IO_L10P_CC_17)
- net IO_L10N_CC_17: now reaches U1.AD20 (IO_L10N_CC_17)
- net IO_L11N_CC_17: now reaches U1.AD21 (IO_L11N_CC_17)
- net IO_L5N_17: now reaches U1.AD23 (IO_L5N_17)
- net IO_L1N_17: now reaches U1.AD24 (IO_L1N_17)
- net IO_L1P_17: now reaches U1.AD25 (IO_L1P_17)
- net IO_L0N_17: now reaches U1.AD26 (IO_L0N_17)
- net IO_L14N_VREF_16: now reaches U1.A3 (IO_L14N_VREF_16)
- net IO_L14N_VREF_16: now also J3.3 (Pin_3)
- net IO_L12N_VRP_16: now reaches U1.A5 (IO_L12N_VRP_16)
- net IO_L10P_CC_16: now reaches U1.A7 (IO_L10P_CC_16)
- net IO_L4N_VREF_16: now reaches U1.A8 (IO_L4N_VREF_16)
- net IO_L4P_16: now reaches U1.A9 (IO_L4P_16)
- net IO_L16N_16: now reaches U1.B5 (IO_L16N_16)
- net IO_L12P_VRN_16: now reaches U1.B6 (IO_L12P_VRN_16)
- net IO_L10N_CC_16: now reaches U1.B7 (IO_L10N_CC_16)
- net IO_L6P_16: now reaches U1.B9 (IO_L6P_16)
- net IO_L9N_CC_16: now reaches U1.C6 (IO_L9N_CC_16)
- net IO_L9P_CC_16: now reaches U1.C7 (IO_L9P_CC_16)
- net IO_L6N_16: now reaches U1.C8 (IO_L6N_16)
- net IO_L8P_CC_16: now reaches U1.C9 (IO_L8P_CC_16)
- net IO_L18P_16: now reaches U1.D5 (IO_L18P_16)
- net IO_L7N_16: now reaches U1.D6 (IO_L7N_16)
- net IO_L8N_CC_16: now reaches U1.D8 (IO_L8N_CC_16)
- net IO_L11P_CC_16: now reaches U1.D9 (IO_L11P_CC_16)
- net IO_L18N_16: now reaches U1.E5 (IO_L18N_16)
- net IO_L5P_12: now reaches U1.G4 (IO_L5P_12)
- net IO_L3P_12: now reaches U1.G5 (IO_L3P_12)
- net IO_L1P_12: now reaches U1.G6 (IO_L1P_12)
- net IO_L5N_12: now reaches U1.H4 (IO_L5N_12)
- net IO_L7P_12: now reaches U1.J5 (IO_L7P_12)
- net IO_L7N_12: now reaches U1.J6 (IO_L7N_12)
- net IO_L9P_CC_12: now reaches U1.K5 (IO_L9P_CC_12)
- net IO_L10P_CC_12: now reaches U1.K6 (IO_L10P_CC_12)
- net IO_L9N_CC_12: now reaches U1.L5 (IO_L9N_CC_12)
- net IO_L9P_CC_18: now reaches U1.AA5 (IO_L9P_CC_18)
- net IO_L9N_CC_18: now reaches U1.AB5 (IO_L9N_CC_18)
- net IO_L10P_CC_18: now reaches U1.AB6 (IO_L10P_CC_18)
- net IO_L10N_CC_18: now reaches U1.AB7 (IO_L10N_CC_18)
- net IO_L19P_18: now reaches U1.AB9 (IO_L19P_18)
- net IO_L12P_VRN_18: now reaches U1.AC6 (IO_L12P_VRN_18)
- net IO_L16N_18: now reaches U1.AC7 (IO_L16N_18)
- net IO_L17N_18: now reaches U1.AC8 (IO_L17P_18)
- net IO_L17N_18: now also U1.AD8 (IO_L17N_18)
- net IO_L18N_18: now reaches U1.AC9 (IO_L18N_18)
- net IO_L14N_VREF_18: now reaches U1.AD4 (IO_L14N_VREF_18)
- net IO_L12N_VRP_18: now reaches U1.AD5 (IO_L12N_VRP_18)
- net IO_L16P_18: now reaches U1.AD6 (IO_L16P_18)
- net IO_L18P_18: now reaches U1.AD9 (IO_L18P_18)
- net IO_L13P_16: now reaches U1.B10 (IO_L13P_16)
- net IO_L15P_16: now reaches U1.B11 (IO_L15P_16)
- net IO_L17P_16: now reaches U1.B12 (IO_L17P_16)
- net IO_L1P_15: now reaches U1.B14 (IO_L1P_15)
- net IO_L3P_15: now reaches U1.B15 (IO_L3P_15)
- net IO_L4P_15: now reaches U1.B16 (IO_L4P_15)
- net IO_L5P_15: now reaches U1.B17 (IO_L5P_15)
- net IO_L7P_15: now reaches U1.B19 (IO_L7P_15)
- net IO_L8N_CC_15: now reaches U1.B20 (IO_L8N_CC_15)
- net IO_L11P_CC_15: now reaches U1.B21 (IO_L11P_CC_15)
- net IO_L13P_15: now reaches U1.B22 (IO_L13P_15)
- net IO_L13P_15: now also U1.B24 (IO_L15P_15)
- net IO_L17P_15: now reaches U1.B25 (IO_L17P_15)
- net IO_L18P_15: now reaches U1.B26 (IO_L18P_15)
- net IO_L0P_15: now reaches U1.C13 (IO_L0P_15)
- net IO_L0N_15: now reaches U1.C14 (IO_L0N_15)
- net IO_L7N_15: now reaches U1.C18 (IO_L7N_15)
- net IO_L11N_CC_15: now reaches U1.C21 (IO_L11N_CC_15)
- net IO_L12N_VRP_15: now reaches U1.C22 (IO_L12N_VRP_15)
- net IO_L15N_15: now reaches U1.C23 (IO_L15N_15)
- net IO_L18N_15: now reaches U1.C26 (IO_L18N_15)
- removed net J5PIN1: J3.2 (Pin_2), J3.3 (Pin_3), J3.4 (Pin_4), J5.1 (Pin_1)
Other:
- moved on the sheet: J1, J4, J5, J6, J7, J8

Commit message: routing
Connections:
- net IO_L13P_15: no longer U1.B24 (IO_L15P_15)
- new net IO_L15P_15: U1.B24 (IO_L15P_15)
Changed lines of the file:
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@@
 		)
 	)
-	(global_label "IO_L13P_15"
+	(global_label "IO_L15P_15"
 		(shape bidirectional)
 		(at 496.57 113.03 0)

Commit message: more routing
Connections:
- net GND: now also J3.22 (Pin_22), J3.23 (Pin_23), J3.29 (Pin_29); no longer J3.21 (Pin_21), J3.35 (Pin_35)
- net VCCO: now also J3.24 (Pin_24), J3.25 (Pin_25), J3.26 (Pin_26), J3.27 (Pin_27)
- net vccext: now reaches J3.30 (Pin_30)
- net vccext: now also J3.31 (Pin_31), J3.32 (Pin_32), J3.33 (Pin_33), J3.34 (Pin_34), J3.35 (Pin_35)

Commit message: more i/o routing and labels
Connections:
- net GND: now also J4.2 (Pin_2), J4.3 (Pin_3), J4.4 (Pin_4), J4.5 (Pin_5), J4.6 (Pin_6); no longer J3.22 (Pin_22)
- net IO_L0N_11: now also J5.12 (Pin_12)
- net IO_L0N_15: now also J4.9 (Pin_9)
- net IO_L0P_11: now also J5.16 (Pin_16)
- net IO_L0P_15: now also J4.8 (Pin_8)
- net IO_L10N_CC_16: now also J3.5 (Pin_5)
- net IO_L10P_CC_15: now also J4.24 (Pin_24)
- net IO_L10P_CC_16: now also J3.6 (Pin_6)
- net IO_L10P_CC_SM15P_11: now also J2.4 (Pin_4)
- net IO_L11N_CC_15: now also J4.31 (Pin_31)
- net IO_L11P_CC_15: now also J4.26 (Pin_26)
- net IO_L11P_CC_16: now also J3.16 (Pin_16)
- net IO_L12N_VRP_11: now also J5.26 (Pin_26)
- net IO_L12N_VRP_15: now also J4.33 (Pin_33)
- net IO_L12N_VRP_16: now also J3.3 (Pin_3)
- net IO_L12P_VRN_15: now also J5.10 (Pin_10)
- net IO_L12P_VRN_16: now also J3.4 (Pin_4)
- net IO_L13N_11: now also J5.29 (Pin_29)
- net IO_L13N_15: now also J4.27 (Pin_27)
- net IO_L13N_16: now also J3.17 (Pin_17)
- net IO_L13P_11: now also J5.27 (Pin_27)
- net IO_L13P_15: now also J4.29 (Pin_29)
- net IO_L13P_16: now also J3.18 (Pin_18)
- net IO_L14N_VREF_11: now also J2.2 (Pin_2)
- net IO_L14N_VREF_15: now also J4.32 (Pin_32)
- net IO_L14N_VREF_16: no longer J3.3 (Pin_3)
- net IO_L14P_11: now also J5.32 (Pin_32)
- net IO_L14P_15: now also J4.30 (Pin_30)
- net IO_L14P_16: now also J1.2 (Pin_2); no longer J3.5 (Pin_5), J3.6 (Pin_6)
- net IO_L15N_15: now also J5.6 (Pin_6)
- net IO_L15N_16: now also J3.20 (Pin_20)
- net IO_L15N_SM13N_11: now also J5.31 (Pin_31)
- net IO_L15P_15: now also J5.2 (Pin_2)
- net IO_L15P_16: now also J3.19 (Pin_19)
- net IO_L15P_CC_SM13P_11: now also J5.34 (Pin_34)
- net IO_L16N_15: now also J5.11 (Pin_11), J5.4 (Pin_4)
- net IO_L16N_16: now also J3.2 (Pin_2)
- net IO_L16N_SM12N_11: now also J2.6 (Pin_6)
- net IO_L16P_16: no longer J3.4 (Pin_4)
- net IO_L17N_15: now also J4.34 (Pin_34)
- net IO_L17N_SM11N_11: now also J2.3 (Pin_3)
- net IO_L17P_15: now also J5.3 (Pin_3)
- net IO_L17P_16: now also J3.21 (Pin_21)
- net IO_L18N_15: now also J5.8 (Pin_8)
- net IO_L18P_15: now also J5.5 (Pin_5)
- net IO_L19N_15: now also J5.9 (Pin_9)
- net IO_L19P_15: now also J5.15 (Pin_15)
- net IO_L1N_11: now also J5.24 (Pin_24)
- net IO_L1N_15: now also J3.22 (Pin_22)
- net IO_L1P_11: now also J5.17 (Pin_17)
- net IO_L1P_15: now also J4.11 (Pin_11)
- net IO_L2N_11: now also J5.23 (Pin_23)
- net IO_L2N_15: now also J4.12 (Pin_12)
- net IO_L2P_15: now also J4.10 (Pin_10)
- net IO_L3N_11: now also J5.19 (Pin_19)
- net IO_L3P_11: now also J5.20 (Pin_20)
- net IO_L3P_15: now also J4.13 (Pin_13)
- net IO_L4N_VREF_16: now also J3.10 (Pin_10)
- net IO_L4P_11: now also J5.13 (Pin_13)
- net IO_L4P_15: now also J4.15 (Pin_15)
- net IO_L4P_16: now also J3.13 (Pin_13)
- net IO_L5N_15: now also J4.16 (Pin_16)
- net IO_L5P_15: now also J4.17 (Pin_17)
- net IO_L6N_15: now also J4.20 (Pin_20)
- net IO_L6N_16: now also J3.9 (Pin_9)
- net IO_L6P_11: now also J5.18 (Pin_18)
- net IO_L6P_15: now also J4.18 (Pin_18)
- net IO_L6P_16: now also J3.12 (Pin_12)
- net IO_L7N_11: now also J5.22 (Pin_22)
- net IO_L7N_15: now also J4.19 (Pin_19)
- net IO_L7N_16: now also J1.4 (Pin_4)
- net IO_L7P_15: now also J4.22 (Pin_22)
- net IO_L7P_16: no longer J3.2 (Pin_2)
- net IO_L8N_CC_15: now also J4.25 (Pin_25)
- net IO_L8N_CC_16: now also J3.11 (Pin_11)
- net IO_L8P_CC_15: now also J4.23 (Pin_23)
- net IO_L8P_CC_16: now also J3.15 (Pin_15)
- net IO_L9N_CC_11: now also J5.30 (Pin_30)
- net IO_L9N_CC_16: now also J1.3 (Pin_3)
- net IO_L9P_CC_11: now also J5.33 (Pin_33)
- net IO_L9P_CC_16: now also J3.8 (Pin_8)
- net IO_L2P_11: now reaches U1.H26 (IO_L2P_11)
- net IO_L2P_11: now also J5.25 (Pin_25)
- net IO_L18P_CC_SM10P_11: now reaches J2.5 (Pin_5)
- net IO_L16P_SM12P_11: now reaches J2.8 (Pin_8)

Commit message: more routing
almost done routing to pins
Connections:
- net IO_L13_N_12 is gone; now on net IO_L13N_12: U1.R5 (IO_L13N_12)
- net IO_L15_N_12 is gone; now on net IO_L15P_12: U1.R6 (IO_L15P_12)
- net IO_L18P_CC_SM10P_11 is gone; now on net IO_L0N_12: J2.5 (Pin_5)
- net IO_L19_N_12 is gone; now on net IO_L19N_12: U1.R7 (IO_L19N_12)
- net GND: now also J3.24 (Pin_24), J3.25 (Pin_25), J3.26 (Pin_26), J3.27 (Pin_27); no longer J3.23 (Pin_23)
- net IO_L0N_17: now also J8.11 (Pin_11)
- net IO_L0N_18: now also J7.30 (Pin_30)
- net IO_L0N_SM8N_13: now also J6.16 (Pin_16)
- net IO_L0P_12: now also J2.6 (Pin_6)
- net IO_L0P_17: now also J8.10 (Pin_10); no longer U1.AF13 (IO_L18P_17)
- net IO_L0P_18: now also J7.29 (Pin_29)
- net IO_L0P_SM8P_13: now also J6.11 (Pin_11)
- net IO_L10N_CC_16: now also J3.6 (Pin_6); no longer J3.5 (Pin_5)
- net IO_L10N_CC_17: now also J8.31 (Pin_31)
- net IO_L10P_CC_12: now also J1.19 (Pin_19)
- net IO_L10P_CC_16: now also J3.8 (Pin_8); no longer J3.6 (Pin_6)
- net IO_L10P_CC_17: now also J7.2 (Pin_2)
- net IO_L10P_CC_18: now also J2.10 (Pin_10)
- net IO_L11N_CC_12: now also J1.32 (Pin_32)
- net IO_L11N_CC_13: now also J6.34 (Pin_34)
- net IO_L11N_CC_17: now also J8.22 (Pin_22)
- net IO_L11N_CC_18: now also J2.23 (Pin_23)
- net IO_L11P_CC_16: now also J3.17 (Pin_17); no longer J3.16 (Pin_16)
- net IO_L11P_CC_17: now also J8.30 (Pin_30)
- net IO_L11P_CC_18: now also J2.29 (Pin_29)
- net IO_L12N_VRP_13: now also J8.2 (Pin_2)
- net IO_L12N_VRP_16: now also J3.4 (Pin_4); no longer J3.3 (Pin_3)
- net IO_L12N_VRP_17: now also J7.12 (Pin_12)
- net IO_L12N_VRP_18: now also J2.11 (Pin_11), J2.18 (Pin_18)
- net IO_L12P_VRN_13: now also J6.33 (Pin_33)
- net IO_L12P_VRN_16: now also J3.5 (Pin_5); no longer J3.4 (Pin_4)
- net IO_L12P_VRN_17: now also J7.6 (Pin_6)
- net IO_L12P_VRN_18: now also J2.25 (Pin_25)
- net IO_L13N_13: now also J8.5 (Pin_5)
- net IO_L13N_16: now also J3.18 (Pin_18); no longer J3.17 (Pin_17)
- net IO_L13N_17: now also J7.4 (Pin_4)
- net IO_L13N_18: now also J2.20 (Pin_20)
- net IO_L13P_12: now also J1.31 (Pin_31)
- net IO_L13P_13: now also J8.3 (Pin_3)
- net IO_L13P_16: now also J3.19 (Pin_19); no longer J3.18 (Pin_18)
- net IO_L13P_17: now also J7.5 (Pin_5)
- net IO_L13P_18: now also J2.17 (Pin_17)
- net IO_L14N_VREF_11: now also J6.2 (Pin_2); no longer J2.2 (Pin_2)
- net IO_L14N_VREF_13: now also J8.8 (Pin_8)
- net IO_L14N_VREF_16: now also J1.5 (Pin_5)
- net IO_L14N_VREF_17: now also J7.13 (Pin_13)
- net IO_L14N_VREF_18: now also J2.13 (Pin_13)
- net IO_L14P_11: now also J5.30 (Pin_30); no longer J5.32 (Pin_32)
- net IO_L14P_13: now also J8.4 (Pin_4)
- net IO_L14P_17: now also J7.10 (Pin_10)
- net IO_L14P_18: now also J2.12 (Pin_12)
- net IO_L15N_12: now also J1.29 (Pin_29)
- net IO_L15N_16: now also J3.21 (Pin_21); no longer J3.20 (Pin_20)
- net IO_L15N_17: now also J7.8 (Pin_8)
- net IO_L15N_18: now also J2.15 (Pin_15)
- net IO_L15N_SM13N_11: now also J5.32 (Pin_32); no longer J5.31 (Pin_31)
- net IO_L15P_13: now also J8.6 (Pin_6)
- net IO_L15P_16: now also J3.20 (Pin_20); no longer J3.19 (Pin_19)
- net IO_L15P_17: now also J7.11 (Pin_11)
- net IO_L15P_18: now also J2.19 (Pin_19)
- net IO_L16N_15: no longer J5.11 (Pin_11), U1.D24 (IO_L16P_15)
- net IO_L16N_16: now also J3.3 (Pin_3); no longer J3.2 (Pin_2)
- net IO_L16N_17: now also J7.18 (Pin_18)
- net IO_L16N_18: now also J2.26 (Pin_26)
- net IO_L16N_SM12N_11: now also J6.6 (Pin_6); no longer J2.6 (Pin_6)
- net IO_L16P_16: now also J1.4 (Pin_4)
- net IO_L16P_17: now also J7.17 (Pin_17)
- net IO_L16P_18: now also J2.16 (Pin_16)
- net IO_L16P_SM12P_11: now also J6.9 (Pin_9), U1.N26 (IO_L16P_SM12P_11); no longer J2.8 (Pin_8)
- net IO_L17N_17: now also J7.15 (Pin_15)
- net IO_L17N_18: now also J2.22 (Pin_22); no longer U1.AC8 (IO_L17P_18)
- net IO_L17N_SM11N_11: now also J6.3 (Pin_3); no longer J2.3 (Pin_3)
- net IO_L17P_12: now also J1.20 (Pin_20)
- net IO_L17P_16: now also J3.22 (Pin_22); no longer J3.21 (Pin_21)
- net IO_L17P_17: now also J7.16 (Pin_16)
- net IO_L17P_SM11P_11: now also J6.4 (Pin_4)
- net IO_L18N_16: now also J1.9 (Pin_9)
- net IO_L18N_17: now also J7.24 (Pin_24)
- net IO_L18N_18: now also J2.33 (Pin_33)
- net IO_L18N_SM10N_11: now also J6.10 (Pin_10)
- net IO_L18P_16: now also J1.8 (Pin_8)
- net IO_L18P_18: now also J2.30 (Pin_30)
- net IO_L18P_SM10P_11: now also J6.5 (Pin_5)
- net IO_L19N_17: now also J7.20 (Pin_20)
- net IO_L19N_SM9N_11: now also J6.8 (Pin_8)
- net IO_L19P_17: now also J7.26 (Pin_26)
- net IO_L19P_SM9P_11: now also J6.12 (Pin_12)
- net IO_L1N_15: now also J3.23 (Pin_23); no longer J3.22 (Pin_22)
- net IO_L1N_17: now also J8.17 (Pin_17)
- net IO_L1N_SM7N_13: now also J6.18 (Pin_18)
- net IO_L1P_12: now also J1.13 (Pin_13)
- net IO_L1P_17: now also J8.13 (Pin_13)
- net IO_L1P_SM7P_13: now also J6.13 (Pin_13)
- net IO_L2N_12: now also J1.34 (Pin_34)
- net IO_L2N_17: now also J8.12 (Pin_12)
- net IO_L2P_12: now also J2.2 (Pin_2)
- net IO_L2P_17: now also J8.16 (Pin_16)
- net IO_L2P_18: now also J7.31 (Pin_31)
- net IO_L2P_SM6P_13: now also J6.15 (Pin_15)
- net IO_L3N_17: now also J8.18 (Pin_18)
- net IO_L3N_SM5N_13: now also J6.19 (Pin_19)
- net IO_L3P_12: now also J1.12 (Pin_12)
- net IO_L3P_17: now also J8.15 (Pin_15)
- net IO_L3P_GC_D9_4: now also J7.33 (Pin_33)
- net IO_L3P_SM5P_13: now also J6.17 (Pin_17)
- net IO_L4N_GC_VREF_4: now also J8.32 (Pin_32)
- net IO_L4N_VREF_12: now also J2.3 (Pin_3)
- net IO_L4N_VREF_13: now also J6.29 (Pin_29)
- net IO_L4N_VREF_16: now also J3.11 (Pin_11); no longer J3.10 (Pin_10)
- net IO_L4N_VREF_17: now also J8.19 (Pin_19)
- net IO_L4N_VREF_18: now also J2.34 (Pin_34)
- net IO_L4P_12: now also J2.4 (Pin_4)
- net IO_L4P_13: now also J6.24 (Pin_24)
- net IO_L4P_16: now also J3.15 (Pin_15); no longer J3.13 (Pin_13)
- net IO_L4P_17: now also J8.23 (Pin_23)
- net IO_L4P_18: now also J2.32 (Pin_32)
- net IO_L5N_17: now also J8.24 (Pin_24)
- net IO_L5N_GC_4: now also J7.25 (Pin_25)
- net IO_L5N_SM4N_13: now also J6.22 (Pin_22)
- net IO_L5P_12: now also J1.11 (Pin_11)
- net IO_L5P_17: now also J8.25 (Pin_25)
- net IO_L5P_GC_4: now also J7.27 (Pin_27)
- net IO_L5P_SM4P_13: now also J6.26 (Pin_26)
- net IO_L6N_16: now also J3.10 (Pin_10); no longer J3.9 (Pin_9)
- net IO_L6N_17: now also J8.20 (Pin_20)
- net IO_L6N_18: now also J7.32 (Pin_32)
- net IO_L6N_D6_2: now also J7.23 (Pin_23)
- net IO_L6P_12: now also J1.33 (Pin_33)
- net IO_L6P_17: now also J8.9 (Pin_9)
- net IO_L6P_18: now also J7.34 (Pin_34)
- net IO_L6P_GC_4: now also J8.34 (Pin_34)
- net IO_L6P_SM3P_13: now also J6.23 (Pin_23)
- net IO_L7N_12: now also J1.15 (Pin_15)
- net IO_L7N_16: now also J1.3 (Pin_3); no longer J1.4 (Pin_4)
- net IO_L7N_GC_VRP: now also J7.19 (Pin_19)
- net IO_L7N_SM2N_13: now also J6.27 (Pin_27)
- net IO_L7P_12: now also J1.16 (Pin_16)
- net IO_L7P_16: now also J1.6 (Pin_6); no longer U1.F5 (IO_L3N_12)
- net IO_L7P_17: now also J8.26 (Pin_26)
- net IO_L7P_GC_VRN_4: now also J7.22 (Pin_22)
- net IO_L8N_CC_16: now also J3.13 (Pin_13); no longer J3.11 (Pin_11)
- net IO_L8N_CC_17: now also J8.27 (Pin_27)
- net IO_L8N_CC_18: now also J2.27 (Pin_27)
- net IO_L8N_CC_SM1N_13: now also J6.32 (Pin_32)
- net IO_L8P_CC_16: now also J3.16 (Pin_16); no longer J3.15 (Pin_15)
- net IO_L8P_CC_17: now also J8.29 (Pin_29)
- net IO_L8P_CC_18: now also J2.24 (Pin_24)
- net IO_L8P_CC_GC_4: now also J7.9 (Pin_9)
- net IO_L8P_CC_SM1P_13: now also J6.31 (Pin_31)
- net IO_L9N_CC_11: now also J5.31 (Pin_31); no longer J5.30 (Pin_30)
- net IO_L9N_CC_12: now also J1.18 (Pin_18)
- net IO_L9N_CC_16: now also J3.2 (Pin_2); no longer J1.3 (Pin_3)
- net IO_L9N_CC_17: now also J8.33 (Pin_33)
- net IO_L9N_CC_18: now also J2.9 (Pin_9)
- net IO_L9P_CC_12: now also J1.17 (Pin_17)
- net IO_L9P_CC_16: now also J3.9 (Pin_9); no longer J3.8 (Pin_8)
- net IO_L9P_CC_17: now also J7.3 (Pin_3)
- net IO_L9P_CC_18: now also J2.8 (Pin_8)
- net IO_L9P_CC_SM0P_13: now also J6.30 (Pin_30)
- net VCCO: no longer J3.24 (Pin_24), J3.25 (Pin_25), J3.26 (Pin_26), J3.27 (Pin_27)
- net IO_L16N_12: now reaches U1.N6 (IO_L16N_12)
- net IO_L16N_12: now also J1.22 (Pin_22)
- net IO_L17N_12: now reaches U1.N7 (IO_L17N_12)
- net IO_L17N_12: now also J1.24 (Pin_24)
- net IO_L16P_12: now reaches U1.P6 (IO_L16P_12)
- net IO_L16P_12: now also J1.23 (Pin_23)
- net IO_L11P_CC_12: now reaches U1.U6 (IO_L11P_CC_12)
- net IO_L11P_CC_12: now also J1.30 (Pin_30)
- net IO_L17N_13: now reaches U1.U22 (IO_L17N_13)
- net IO_L17N_13: now also J6.20 (Pin_20)
- net IO_L18N_13: now reaches U1.V22 (IO_L18N_13)
- net IO_L18N_13: now also J6.25 (Pin_25)
- net IO_L3N_12: now reaches J1.10 (Pin_10)
- net IO_L3N_12: now also U1.F5 (IO_L3N_12)
- net IO_L15P_12: now reaches J1.25 (Pin_25)
- net IO_L19N_12: now reaches J1.26 (Pin_26)
- net IO_L13N_12: now reaches J1.27 (Pin_27)
- net IO_L17P_18: now reaches J2.31 (Pin_31)
- net IO_L17P_18: now also U1.AC8 (IO_L17P_18)
- net IO_L10N_CC_18: no longer names the net of U1.AB7 (IO_L10N_CC_18)
- net IO_L10N_CC_SM15N_11: no longer names the net of U1.L22 (IO_L10N_CC_SM15N_11)
- net IO_L10P_CC_SM15P_11: no longer names the net of U1.L23 (IO_L10P_CC_SM15P_11)
- net IO_L10P_CC_SM15P_11: no longer J2.4 (Pin_4)
- net IO_L19P_18: no longer names the net of U1.AB9 (IO_L19P_18)
- net IO_L2N_SM6N_13: no longer names the net of U1.P23 (IO_L2N_SM6N_13)
- net IO_L5N_12: no longer names the net of U1.H4 (IO_L5N_12)
- net IO_L6N_11: no longer names the net of U1.H22 (IO_L6N_11)
- new net IO_L16P_15: J5.11 (Pin_11), U1.D24 (IO_L16P_15)
- new net IO_L18P_17: U1.AF13 (IO_L18P_17)
Other:
- moved on the sheet: J1, J2, J3, J4, J5, J6, J7, J8

Commit message: more routing
Connections:
- net GND: no longer J3.24 (Pin_24), J3.25 (Pin_25)
- net IO_L0N_12: now also J2.3 (Pin_3); no longer J2.5 (Pin_5)
- net IO_L0N_18: now also J7.33 (Pin_33); no longer J7.30 (Pin_30)
- net IO_L0P_12: now also J2.4 (Pin_4); no longer J2.6 (Pin_6)
- net IO_L0P_18: now also J7.32 (Pin_32); no longer J7.29 (Pin_29)
- net IO_L10N_CC_16: now also J3.9 (Pin_9); no longer J3.6 (Pin_6)
- net IO_L10P_CC_12: now also J1.17 (Pin_17); no longer J1.19 (Pin_19)
- net IO_L10P_CC_16: now also J3.10 (Pin_10); no longer J3.8 (Pin_8)
- net IO_L10P_CC_18: now also J2.8 (Pin_8); no longer J2.10 (Pin_10)
- net IO_L11N_CC_12: now also J1.30 (Pin_30); no longer J1.32 (Pin_32)
- net IO_L11N_CC_18: now also J2.20 (Pin_20); no longer J2.23 (Pin_23)
- net IO_L11P_CC_12: now also J1.27 (Pin_27); no longer J1.30 (Pin_30)
- net IO_L11P_CC_16: now also J3.25 (Pin_25); no longer J3.17 (Pin_17)
- net IO_L11P_CC_18: now also J2.26 (Pin_26); no longer J2.29 (Pin_29)
- net IO_L12N_VRP_16: now also J3.6 (Pin_6); no longer J3.4 (Pin_4)
- net IO_L12N_VRP_18: now also J2.9 (Pin_9); no longer J2.11 (Pin_11), J2.18 (Pin_18)
- net IO_L12P_VRN_16: now also J3.8 (Pin_8); no longer J3.5 (Pin_5)
- net IO_L12P_VRN_18: now also J2.23 (Pin_23); no longer J2.25 (Pin_25)
- net IO_L13N_12: now also J1.25 (Pin_25); no longer J1.27 (Pin_27)
- net IO_L13N_16: now also J3.19 (Pin_19); no longer J3.18 (Pin_18)
- net IO_L13N_18: now also J2.18 (Pin_18); no longer J2.20 (Pin_20)
- net IO_L13P_12: now also J1.29 (Pin_29); no longer J1.31 (Pin_31)
- net IO_L13P_16: now also J3.20 (Pin_20); no longer J3.19 (Pin_19)
- net IO_L13P_18: now also J2.15 (Pin_15); no longer J2.17 (Pin_17)
- net IO_L14N_VREF_16: now also J1.3 (Pin_3); no longer J1.5 (Pin_5)
- net IO_L14N_VREF_18: now also J2.11 (Pin_11); no longer J2.13 (Pin_13)
- net IO_L14P_16: now also J3.3 (Pin_3); no longer J1.2 (Pin_2)
- net IO_L14P_18: now also J2.10 (Pin_10); no longer J2.12 (Pin_12)
- net IO_L15N_12: now also J1.26 (Pin_26); no longer J1.29 (Pin_29)
- net IO_L15N_16: now also J3.22 (Pin_22); no longer J3.21 (Pin_21)
- net IO_L15N_18: now also J2.12 (Pin_12); no longer J2.15 (Pin_15)
- net IO_L15P_12: now also J1.23 (Pin_23); no longer J1.25 (Pin_25)
- net IO_L15P_16: now also J3.21 (Pin_21); no longer J3.20 (Pin_20)
- net IO_L15P_18: now also J2.17 (Pin_17); no longer J2.19 (Pin_19)
- net IO_L16N_12: now also J1.19 (Pin_19); no longer J1.22 (Pin_22)
- net IO_L16N_16: now also J3.5 (Pin_5); no longer J3.3 (Pin_3)
- net IO_L16N_18: now also J2.24 (Pin_24); no longer J2.26 (Pin_26)
- net IO_L16P_12: now also J1.20 (Pin_20); no longer J1.23 (Pin_23)
- net IO_L16P_16: now also J1.2 (Pin_2); no longer J1.4 (Pin_4)
- net IO_L16P_18: now also J2.13 (Pin_13); no longer J2.16 (Pin_16)
- net IO_L17N_12: now also J1.22 (Pin_22); no longer J1.24 (Pin_24)
- net IO_L17N_18: now also J2.19 (Pin_19); no longer J2.22 (Pin_22)
- net IO_L17P_12: now also J1.18 (Pin_18); no longer J1.20 (Pin_20)
- net IO_L17P_16: now also J3.23 (Pin_23); no longer J3.22 (Pin_22)
- net IO_L17P_18: now also J2.29 (Pin_29); no longer J2.31 (Pin_31)
- net IO_L18N_16: now also J1.6 (Pin_6); no longer J1.9 (Pin_9)
- net IO_L18N_18: now also J2.31 (Pin_31); no longer J2.33 (Pin_33)
- net IO_L18P_16: now also J1.5 (Pin_5); no longer J1.8 (Pin_8)
- net IO_L18P_17: now also J7.30 (Pin_30)
- net IO_L18P_18: now also J2.27 (Pin_27); no longer J2.30 (Pin_30)
- net IO_L19N_12: now also J1.24 (Pin_24); no longer J1.26 (Pin_26)
- net IO_L1N_15: now also J3.24 (Pin_24); no longer J3.23 (Pin_23)
- net IO_L1P_12: now also J1.11 (Pin_11); no longer J1.13 (Pin_13)
- net IO_L2N_12: now also J1.32 (Pin_32); no longer J1.34 (Pin_34)
- net IO_L2N_18: now also J7.27 (Pin_27)
- net IO_L2P_12: now also J1.33 (Pin_33); no longer J2.2 (Pin_2)
- net IO_L2P_18: now also J7.34 (Pin_34); no longer J7.31 (Pin_31)
- net IO_L3N_12: now also J1.8 (Pin_8); no longer J1.10 (Pin_10)
- net IO_L3P_12: now also J1.10 (Pin_10); no longer J1.12 (Pin_12)
- net IO_L3P_GC_D9_4: now also J7.31 (Pin_31); no longer J7.33 (Pin_33)
- net IO_L4N_VREF_12: now also J1.34 (Pin_34); no longer J2.3 (Pin_3)
- net IO_L4N_VREF_16: now also J3.13 (Pin_13); no longer J3.11 (Pin_11)
- net IO_L4N_VREF_18: now also J2.32 (Pin_32); no longer J2.34 (Pin_34)
- net IO_L4P_12: now also J2.2 (Pin_2); no longer J2.4 (Pin_4)
- net IO_L4P_16: now also J3.16 (Pin_16); no longer J3.15 (Pin_15)
- net IO_L4P_18: now also J2.30 (Pin_30); no longer J2.32 (Pin_32)
- net IO_L5P_12: now also J1.9 (Pin_9); no longer J1.11 (Pin_11)
- net IO_L5P_GC_4: now also J7.29 (Pin_29); no longer J7.27 (Pin_27)
- net IO_L6N_16: now also J3.12 (Pin_12); no longer J3.10 (Pin_10)
- net IO_L6N_18: now also J2.34 (Pin_34); no longer J7.32 (Pin_32)
- net IO_L6P_12: now also J1.31 (Pin_31); no longer J1.33 (Pin_33)
- net IO_L6P_16: now also J3.15 (Pin_15); no longer J3.12 (Pin_12)
- net IO_L6P_18: now also J2.33 (Pin_33); no longer J7.34 (Pin_34)
- net IO_L7N_12: now also J1.12 (Pin_12); no longer J1.15 (Pin_15)
- net IO_L7N_16: now also J3.2 (Pin_2); no longer J1.3 (Pin_3)
- net IO_L7P_12: now also J1.13 (Pin_13); no longer J1.16 (Pin_16)
- net IO_L7P_16: now also J1.4 (Pin_4); no longer J1.6 (Pin_6)
- net IO_L8N_CC_16: now also J3.17 (Pin_17); no longer J3.13 (Pin_13)
- net IO_L8N_CC_18: now also J2.25 (Pin_25); no longer J2.27 (Pin_27)
- net IO_L8P_CC_16: now also J3.18 (Pin_18); no longer J3.16 (Pin_16)
- net IO_L8P_CC_18: now also J2.22 (Pin_22); no longer J2.24 (Pin_24)
- net IO_L9N_CC_12: now also J1.16 (Pin_16); no longer J1.18 (Pin_18)
- net IO_L9N_CC_16: now also J3.4 (Pin_4); no longer J3.2 (Pin_2)
- net IO_L9N_CC_18: now also J2.6 (Pin_6); no longer J2.9 (Pin_9)
- net IO_L9P_CC_12: now also J1.15 (Pin_15); no longer J1.17 (Pin_17)
- net IO_L9P_CC_16: now also J3.11 (Pin_11); no longer J3.9 (Pin_9)
- net IO_L9P_CC_18: now also J2.5 (Pin_5); no longer J2.8 (Pin_8)
