File: XC5VLX30T_testboard/XC5VLX30T_testboard.kicad_sch (KiCad schematic)
At the start: 19 parts, among them J1 Conn_01x35_Pin, J2 Conn_01x35_Pin, J3 Conn_01x35_Pin, J4 Conn_01x35_Pin, J5 Conn_01x35_Pin, J6 Conn_01x35_Pin, J7 Conn_01x35_Pin, J8 Conn_01x35_Pin, U1 XC5VLX30T-1FFG665C, X1 SG-5032CCN

Commit message: through hole pads for buck converters
Parts:
- added C5, C9: 470uF, Capacitor_Tantalum_SMD:CP_EIA-3216-12_Kemet-S, symbol Device:C
- added C6: 470uF, Capacitor_Tantalum_SMD:CP_EIA-3216-10_Kemet-I, symbol Device:C
- added J10, J11, J12, J13, J14, J9: Conn_01x04_Pin, Connector_PinHeader_2.54mm:PinHeader_1x04_P2.54mm_Vertical, symbol Connector:Conn_01x04_Pin
- C1: footprint Capacitor_Tantalum_SMD:CP_EIA-3528-12_Kemet-T -> Capacitor_Tantalum_SMD:CP_EIA-3216-10_Kemet-I
- C12, C13, C15, C2, C3, C4, C7, C8: footprint Capacitor_Tantalum_SMD:CP_EIA-3528-12_Kemet-T -> Capacitor_Tantalum_SMD:CP_EIA-3216-12_Kemet-S
- X1: footprint Oscillator:Oscillator_SMD_SeikoEpson_SG8002LB-4Pin_5.0x3.2mm -> Crystal:Crystal_SMD_3225-4Pin_3.2x2.5mm_HandSoldering
Connections:
- net GND: now also C5.2, C6.2, C9.2
- net IO_L10P_CC_12: now also J1.15 (Pin_15); no longer J1.17 (Pin_17)
- net IO_L4N_VREF_16: now also J3.17 (Pin_17); no longer J3.13 (Pin_13)
- net IO_L8N_CC_16: now also J3.13 (Pin_13); no longer J3.17 (Pin_17)
- net IO_L9N_CC_12: now also J1.17 (Pin_17); no longer J1.16 (Pin_16)
- net IO_L9P_CC_12: now also J1.16 (Pin_16); no longer J1.15 (Pin_15)
- net VCCO: now also C9.1, J12.1 (Pin_1), J12.2 (Pin_2), J12.3 (Pin_3), J12.4 (Pin_4)
- net VccAUX: now also C5.1, J10.1 (Pin_1), J10.2 (Pin_2), J10.3 (Pin_3), J10.4 (Pin_4)
- net VccINT: now also C6.1, J14.1 (Pin_1), J14.2 (Pin_2), J14.3 (Pin_3), J14.4 (Pin_4)

Commit message: more clicking
Connections:
- net GND: now also J10.1 (Pin_1), J10.2 (Pin_2), J11.3 (Pin_3), J11.4 (Pin_4), J12.1 (Pin_1), J12.2 (Pin_2), J13.3 (Pin_3), J13.4 (Pin_4), J14.1 (Pin_1), J14.2 (Pin_2), J9.3 (Pin_3), J9.4 (Pin_4)
- net VCCO: no longer J12.1 (Pin_1), J12.2 (Pin_2)
- net VccAUX: no longer J10.1 (Pin_1), J10.2 (Pin_2)
- net VccINT: no longer J14.1 (Pin_1), J14.2 (Pin_2)
- net vccext: now also J11.1 (Pin_1), J11.2 (Pin_2), J13.1 (Pin_1), J13.2 (Pin_2), J9.1 (Pin_1), J9.2 (Pin_2)
