File: XC5VLX30T_testboard/buck_converter_mp2307/buck_converter_mp2307.kicad_sch (KiCad schematic)
At the start: 12 parts, among them J1 Conn_02x01, J4 Conn_01x06_Pin, U1 MP2307DN-LF-Z

Commit message: reordered headers
Parts:
- removed C5: 22uF, Capacitor_SMD:C_0603_1608Metric, symbol Device:C
- removed J1: Conn_02x01, Connector_PinHeader_2.54mm:PinHeader_2x01_P2.54mm_Vertical, symbol Connector_Generic:Conn_02x01
- added C6: 0.1uF, Capacitor_SMD:C_0603_1608Metric, symbol Device:C
- added C8: 22uF, Capacitor_SMD:C_1206_3216Metric, symbol Device:C
- added J2: Inductor L, Connector_PinHeader_2.54mm:PinHeader_1x01_P2.54mm_Vertical, symbol Connector:Conn_01x01_Pin
- added J3: Inductor_R, Connector_PinHeader_2.54mm:PinHeader_1x01_P2.54mm_Vertical, symbol Connector:Conn_01x01_Pin
- C2: footprint Capacitor_SMD:C_0603_1608Metric -> Capacitor_SMD:C_1206_3216Metric
- R1, R2, R3, R4: footprint Resistor_SMD:R_0402_1005Metric -> Resistor_SMD:R_0603_1608Metric
Connections:
- net GND: now also C6.2, C8.2
- net VCCoutput: now also J2.1 (Pin_1)
- net vccext: now also C8.1
- net SWITCHED: now reaches C1.2, U1.3 (SW)
- net SWITCHED: now also J3.1 (Pin_1)
- net at C3.1, U1.6 (COMP): now also C6.1
Other:
- moved on the sheet: J4
